File: RAM2E.kicad_pcb (KiCad board)
At the start: 4 copper layers, 78.2 x 50 mm, 63 parts, among them J1 AppleIIeAux, J2 JTAG, U1 EPM240T100, U2 W9864G6KH-6, U3 74AHC245, U4 74LVC245, U5 74AHC245, U6 74AHCT245, U7 74AHCT245, U8 TPS73701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

Commit message: As submitted to JLCPCB August 2020
Parts:
- removed C30: DNP, stdpads:C_0805
- removed R1: 5k76, stdpads:R_0805
- removed R2: 3k3, stdpads:R_0805
- removed R3, R4, R8: DNP, stdpads:R_0805
- removed R5: 0, stdpads:R_0805
- removed U9: DNP, stdpads:SOT-223-6
- H1, H2, H3, H4: footprint stdpads:PasteHole_1.1mm_PTH -> stdpads:PasteHole_1.152mm_NPTH
- R9: value 1k2 -> 22k
- RN1, RN2, RN3: value 4x100 -> 4x33; footprint stdpads:Yageo_YC124 -> stdpads:R4_0402
- U2: value W9864G6KH-6 -> W9812G6KH-6
- U8: value TPS73701 -> AP2125N-3.3; footprint stdpads:SOT-223-6 -> stdpads:SOT-23
- moved C1 7.98 mm to (271.4, 111.7)
- moved U8 5.92 mm to (267.6, 110.8)
- moved C5 4.88 mm to (261.2, 106.8), turned to 270 degrees
- moved C2 4.72 mm to (266.6, 106.8)
- moved C3 4.55 mm to (261.2, 110.8), turned to 90 degrees
- moved C6 2.52 mm to (263.9, 106.8), turned to 270 degrees
- moved C4 1.79 mm to (263.9, 110.8), turned to 90 degrees
- turned RN1 to 270 degrees
- turned RN2 to 270 degrees
- turned RN3 to 0 degrees
- turned U1 to 270 degrees
- turned U3 to 0 degrees
- turned U4 to 0 degrees
- turned U5 to 0 degrees
- turned U6 to 0 degrees
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Connections:
- net /CFG0 renamed Net-(U1-Pad87)
- net /CFG1 renamed Net-(U1-Pad86)
- net /CFG2 renamed Net-(U1-Pad88)
- C16 pad 1: +1V8 -> +3V3
- C19 pad 1: +1V8 -> +3V3
- C2 pad 1: +5V -> +3V3
- C5 pad 1: +1V8 -> +3V3
- C6 pad 1: +1V8 -> +3V3
- RN3 pad 2: Net-(RN3-Pad1) -> Net-(RN3-Pad2)
- RN3 pad 3: Net-(RN3-Pad1) -> Net-(RN3-Pad3)
- RN3 pad 6: /ACLK -> Net-(RN3-Pad6)
- RN3 pad 7: /RCLK -> Net-(RN3-Pad7)
- U1 pad 13: +1V8 -> +3V3
- U1 pad 63: +1V8 -> +3V3
- U1 pad 82: /DlyIn -> Net-(U1-Pad82)
- U1 pad 83: /DlyOut -> Net-(U1-Pad83)
- U2 pad 36: Net-(U2-Pad36) -> GND
- U8 pad 1: +5V -> GND
- U8 pad 3: GND -> +5V
Routing:
- net +1V8: track 274.5 -> 0.00 mm, vias 16 -> 0
- net +5V: track 227.7 -> 182.4 mm, vias 12 -> 11
- net +3V3: track 102.0 -> 121.6 mm, vias 79 -> 91
- net /DlyIn: track 17.7 -> 0.00 mm, vias 2 -> 0
- net GND: track 177.7 -> 160.7 mm, vias 314 -> 307
- net /DlyOut: track 15.7 -> 0.00 mm, vias 2 -> 0
- net Net-(R3-Pad2): track 4.55 -> 0.00 mm
- net Net-(R1-Pad2): track 4.55 -> 0.00 mm
- net /C14M: track 54.0 -> 55.5 mm
- net /TMS: track 99.3 -> 97.9 mm
- net /TDI: track 86.9 -> 85.5 mm
- net /TCK: track 83.2 -> 81.9 mm
- net /TDO: track 104.6 -> 103.3 mm
- net /RCLK: track 5.78 -> 4.83 mm
- net /~EN80~: track 48.4 -> 49.2 mm
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
Commit message: August 2020 JLCPCB again
Parts:
- moved C24 0.40 mm to (213.8, 118.0)
- moved C25 0.40 mm to (223.8, 118.0)
- moved C20 0.20 mm to (213.8, 93.2)
- moved C28 0.20 mm to (223.8, 93.2)
Routing:
- net GND: track 160.7 -> 162.1 mm, vias 307 -> 308
- net /TDO: track 103.3 -> 104.1 mm
- net +3V3: track 121.6 -> 122.2 mm
