File: RAM2E.kicad_pcb (KiCad board)
At the start: 4 copper layers, 78.2 x 50 mm, 55 parts, among them J1 AppleIIeAux, J2 JTAG, U1 EPM240T100, U2 W9812G6KH-6, U3 74AHC245, U4 74LVC245, U5 74AHC245, U6 74AHCT245, U7 74AHCT245, U8 AP2125N-3.3

Commit message: As submitted to JLCPCB August 21 2020
Connections:
- U4 pad 3: Net-(U4-Pad3) -> GND
- U4 pad 4: Net-(U4-Pad4) -> GND
Changed lines of the file:
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@@
     (zones 0)
     (modules 55)
-    (nets 166)
+    (nets 164)
   )
   (page A4)
@@
   )
   (setup
-    (last_trace_width 0.5)
+    (last_trace_width 0.15)
     (user_trace_width 0.2)
     (user_trace_width 0.25)
@@
   (net 152 "Net-(U4-Pad17)")
   (net 153 "Net-(U4-Pad16)")
-  (net 154 "Net-(U4-Pad4)")
-  (net 155 "Net-(U4-Pad3)")
-  (net 156 /~FRCTXT~)
-  (net 157 "Net-(U1-Pad88)")
-  (net 158 "Net-(U1-Pad87)")
-  (net 159 "Net-(U1-Pad86)")
-  (net 160 "Net-(RN3-Pad3)")
-  (net 161 "Net-(RN3-Pad2)")
-  (net 162 "Net-(RN3-Pad7)")
-  (net 163 "Net-(RN3-Pad6)")
-  (net 164 "Net-(U1-Pad82)")
-  (net 165 "Net-(U1-Pad83)")
+  (net 154 /~FRCTXT~)
+  (net 155 "Net-(U1-Pad88)")
+  (net 156 "Net-(U1-Pad87)")
+  (net 157 "Net-(U1-Pad86)")
+  (net 158 "Net-(RN3-Pad3)")
+  (net 159 "Net-(RN3-Pad2)")
+  (net 160 "Net-(RN3-Pad7)")
+  (net 161 "Net-(RN3-Pad6)")
+  (net 162 "Net-(U1-Pad82)")
+  (net 163 "Net-(U1-Pad83)")
   (net_class Default "This is the default net class."
     (clearance 0.15)
@@
     (add_net "Net-(U4-Pad16)")
     (add_net "Net-(U4-Pad17)")
-    (add_net "Net-(U4-Pad3)")
-    (add_net "Net-(U4-Pad4)")
   )
   (module stdpads:C_0603 (layer F.Cu)
@@
       (net 105 "Net-(U1-Pad81)"))
     (pad 82 smd roundrect (at -7.6625 -3) (size 0.3 1.475) (layers F.Cu F.Paste F.Mask) (roundrect_rratio 0.25)
-      (net 164 "Net-(U1-Pad82)"))
+      (net 162 "Net-(U1-Pad82)"))
     (pad 83 smd roundrect (at -7.6625 -2.5) (size 0.3 1.475) (layers F.Cu F.Paste F.Mask) (roundrect_rratio 0.25)
-      (net 165 "Net-(U1-Pad83)"))
+      (net 163 "Net-(U1-Pad83)"))
     (pad 84 smd roundrect (at -7.6625 -2) (size 0.3 1.475) (layers F.Cu F.Paste F.Mask) (roundrect_rratio 0.25)
       (net 139 /Dout6))
@@
       (net 140 /Dout7))
     (pad 86 smd roundrect (at -7.6625 -1) (size 0.3 1.475) (layers F.Cu F.Paste F.Mask) (roundrect_rratio 0.25)
-      (net 159 "Net-(U1-Pad86)"))
+      (net 157 "Net-(U1-Pad86)"))
     (pad 87 smd roundrect (at -7.6625 -0.5) (size 0.3 1.475) (layers F.Cu F.Paste F.Mask) (roundrect_rratio 0.25)
-      (net 158 "Net-(U1-Pad87)"))
+      (net 156 "Net-(U1-Pad87)"))
     (pad 88 smd roundrect (at -7.6625 0) (size 0.3 1.475) (layers F.Cu F.Paste F.Mask) (roundrect_rratio 0.25)
-      (net 157 "Net-(U1-Pad88)"))
+      (net 155 "Net-(U1-Pad88)"))
     (pad 89 smd roundrect (at -7.6625 0.5) (size 0.3 1.475) (layers F.Cu F.Paste F.Mask) (roundrect_rratio 0.25)
       (net 144 /RD3r))
@@
       (net 151 "Net-(RN3-Pad1)") (solder_paste_margin -0.035))
     (pad 3 smd roundrect (at 0.25 0.5 90) (size 0.65 0.3) (layers F.Cu F.Paste F.Mask) (roundrect_rratio 0.25)
-      (net 160 "Net-(RN3-Pad3)"))
+      (net 158 "Net-(RN3-Pad3)"))
     (pad 2 smd roundrect (at -0.25 0.5 90) (size 0.65 0.3) (layers F.Cu F.Paste F.Mask) (roundrect_rratio 0.25)
-      (net 161 "Net-(RN3-Pad2)"))
+      (net 159 "Net-(RN3-Pad2)"))
     (pad 4 smd roundrect (at 0.8 0.5 90) (size 0.65 0.4) (layers F.Cu F.Paste F.Mask) (roundrect_rratio 0.25)
       (net 151 "Net-(RN3-Pad1)") (solder_paste_margin -0.035))
     (pad 7 smd roundrect (at -0.25 -0.5 90) (size 0.65 0.3) (layers F.Cu F.Paste F.Mask) (roundrect_rratio 0.25)
-      (net 162 "Net-(RN3-Pad7)"))
+      (net 160 "Net-(RN3-Pad7)"))
     (pad 8 smd roundrect (at -0.8 -0.5 90) (size 0.65 0.4) (layers F.Cu F.Paste F.Mask) (roundrect_rratio 0.25)
       (net 149 /RCLK) (solder_paste_margin -0.035))
     (pad 6 smd roundrect (at 0.25 -0.5 90) (size 0.65 0.3) (layers F.Cu F.Paste F.Mask) (roundrect_rratio 0.25)
-      (net 163 "Net-(RN3-Pad6)"))
+      (net 161 "Net-(RN3-Pad6)"))
     (pad 5 smd roundrect (at 0.8 -0.5 90) (size 0.65 0.4) (layers F.Cu F.Paste F.Mask) (roundrect_rratio 0.25)
       (net 150 /ACLK) (solder_paste_margin -0.035))
@@
       (net 30 /~EN80~))
     (pad 4 smd roundrect (at -0.975 2.95 90) (size 1.45 0.45) (layers F.Cu F.Paste F.Mask) (roundrect_rratio 0.25)
-      (net 154 "Net-(U4-Pad4)"))
+      (net 2 GND))
     (pad 3 smd roundrect (at -1.625 2.95 90) (size 1.45 0.45) (layers F.Cu F.Paste F.Mask) (roundrect_rratio 0.25)
-      (net 155 "Net-(U4-Pad3)"))
+      (net 2 GND))
     (pad 2 smd roundrect (at -2.275 2.95 90) (size 1.45 0.45) (layers F.Cu F.Paste F.Mask) (roundrect_rratio 0.25)
       (net 50 /C14M))
@@
       (net 29 /AN3))
     (pad 1 smd roundrect (at -0.95 0) (size 0.85 1.4) (layers F.Cu F.Paste F.Mask) (roundrect_rratio 0.25)
-      (net 156 /~FRCTXT~))
+      (net 154 /~FRCTXT~))
     (model ${KISYS3DMOD}/Resistor_SMD.3dshapes/R_0805_2012Metric.wrl
       (at (xyz 0 0 0))
@@
       (net 29 /AN3))
     (pad 1 smd roundrect (at -0.95 0) (size 0.85 1.4) (layers F.Cu F.Paste F.Mask) (roundrect_rratio 0.25)
-      (net 156 /~FRCTXT~))
+      (net 154 /~FRCTXT~))
   )
   (module stdpads:C_0805 (layer F.Cu)
@@
       (net 37 /~RA9~))
     (pad 55 smd roundrect (at -24.13 -0.1 180) (size 1.524 7.34) (layers B.Cu B.Mask) (roundrect_rratio 0.25)
-      (net 156 /~FRCTXT~))
+      (net 154 /~FRCTXT~))
     (pad 54 smd roundrect (at -21.59 -0.1 180) (size 1.524 7.34) (layers B.Cu B.Mask) (roundrect_rratio 0.25)
       (net 36 /SEGB))
@@
   (segment (start 229.15 111.65) (end 228.4 112.4) (width 0.15) (layer F.Cu) (net 151))
   (segment (start 229.15 111.15) (end 229.15 111.65) (width 0.15) (layer F.Cu) (net 151))
-  (via (at 207.518 124.0155) (size 0.5) (drill 0.2) (layers F.Cu B.Cu) (net 156))
-  (segment (start 208.346 124.0155) (end 207.518 124.0155) (width 0.15) (layer F.Cu) (net 156))
-  (via (at 207.518 126.1745) (size 0.5) (drill 0.2) (layers F.Cu B.Cu) (net 156))
-  (segment (start 208.346 126.1745) (end 207.518 126.1745) (width 0.15) (layer F.Cu) (net 156))
-  (segment (start 207.518 126.1745) (end 207.518 124.0155) (width 0.15) (layer B.Cu) (net 156))
-  (segment (start 208.7245 126.1745) (end 207.518 126.1745) (width 0.15) (layer B.Cu) (net 156))
-  (segment (start 213.36 130.81) (end 208.7245 126.1745) (width 0.15) (layer B.Cu) (net 156))
-  (segment (start 213.36 135.282) (end 213.36 130.81) (width 0.15) (layer B.Cu) (net 156))
+  (via (at 207.518 124.0155) (size 0.5) (drill 0.2) (layers F.Cu B.Cu) (net 154))
+  (segment (start 208.346 124.0155) (end 207.518 124.0155) (width 0.15) (layer F.Cu) (net 154))
+  (via (at 207.518 126.1745) (size 0.5) (drill 0.2) (layers F.Cu B.Cu) (net 154))
+  (segment (start 208.346 126.1745) (end 207.518 126.1745) (width 0.15) (layer F.Cu) (net 154))
+  (segment (start 207.518 126.1745) (end 207.518 124.0155) (width 0.15) (layer B.Cu) (net 154))
+  (segment (start 208.7245 126.1745) (end 207.518 126.1745) (width 0.15) (layer B.Cu) (net 154))
+  (segment (start 213.36 130.81) (end 208.7245 126.1745) (width 0.15) (layer B.Cu) (net 154))
+  (segment (start 213.36 135.282) (end 213.36 130.81) (width 0.15) (layer B.Cu) (net 154))
   (zone (net 2) (net_name GND) (layer F.Cu) (hatch edge 0.508)
     (connect_pads (clearance 0.154))
