File: RAM2E.sch (KiCad schematic (older format))
At the start: 55 parts, among them J1 AppleIIeAux, J2 JTAG, U1 EPM240T100, U2 W9812G6KH-6, U3 74AHC245, U4 74LVC245, U5 74AHC245, U6 74AHCT245, U7 74AHCT245, U8 AP2125N-3.3

Commit message: As submitted to JLCPCB August 21 2020
Connections:
- net GND: now also U4.3 (A1), U4.4 (A2)
Changed lines of the file:
@@
 Wire Wire Line
 	8600 1750 8600 1650
+$Comp
+L power:GND #PWR?
+U 1 1 5F4141A1
+P 2300 2550
+F 0 "#PWR?" H 2300 2300 50  0001 C CNN
+F 1 "GND" H 2300 2400 50  0000 C CNN
+F 2 "" H 2300 2550 50  0001 C CNN
+F 3 "" H 2300 2550 50  0001 C CNN
+	1    2300 2550
+	1    0    0    -1
+$EndComp
+Wire Wire Line
+	2300 2550 2600 2550
+Wire Wire Line
+	2600 2550 2600 2650
 Wire Bus Line
 	8200 4250 8200 5350
+Connection ~ 2600 2550
 $EndSCHEMATC
