File: Hardware/MAX/RAM2E.kicad_pcb (KiCad board)
At the start: 4 copper layers, 78.2 x 50 mm, 62 parts, among them J1 AppleIIeAux, J2 JTAG, J3 C14M, U1 EPM240T100C5N, U2 W9812G6KH-6, U3 74LVC245APW, U4 74LVC245APW, U5 74LVC245APW, U6 74AHCT245PW, U7 74AHCT245PW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

Commit message: started
Parts:
- R1: value 0 -> 0
- U9: value DNP -> AP2127K-1.8TRG1
Changed lines of the file:
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@@
       (effects (font (size 0.254 0.254) (thickness 0.0635)))
     )
-    (fp_text value 0 (at 0 0.35 90) (layer F.Fab)
+    (fp_text value "0 " (at 0 0.35 90) (layer F.Fab)
       (effects (font (size 0.254 0.254) (thickness 0.0635)))
     )
@@
       (effects (font (size 0.381 0.381) (thickness 0.09525)))
     )
-    (fp_text value DNP (at -0.4 0 270) (layer F.Fab)
+    (fp_text value AP2127K-1.8TRG1 (at -0.4 0 270) (layer F.Fab)
       (effects (font (size 0.127 0.127) (thickness 0.03175)))
     )

Commit message: still workin
Connections:
- RN1 pad 8: /RD7r -> /RD0r
- RN2 pad 5: /RD0r -> /RD7r
- U1 pad 96: /RD7r -> /RD0r
- U1 pad 97: /RD0r -> /RD7r
Routing:
- net +5V: track 194.6 -> 214.5 mm, vias 13 -> 16
- net /RD7r: track 9.07 -> 11.1 mm
- net /RD0r: track 11.1 -> 9.07 mm
- net GND: track 161.8 -> 161.6 mm, vias 291 -> 289
