File: Hardware/MAX/RAM2E.kicad_pcb (KiCad board)
At the start: 4 copper layers, 78.2 x 50 mm, 62 parts, among them J1 AppleIIeAux, J2 JTAG, J3 C14M, U1 EPM240T100C5N, U2 W9812G6KH-6, U3 74LVC245APW, U4 74LVC245APW, U5 74LVC245APW, U6 74AHCT245PW, U7 74AHCT245PW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

Commit message: idk
Parts:
- removed RN1, RN2, RN3, RN4, RN5: 4x33, stdpads:R4_0402
- added R4: 47, stdpads:R_0603, F.Cu at (226.8, 119.0)
- added R5: 47, stdpads:R_0603, F.Cu at (228.2, 119.0)
- moved C25 2.05 mm to (223.8, 118.0), turned to 0 degrees
Connections:
- U1 pad 89: /RD3r -> /RD3
- U1 pad 90: /RD1r -> /RD1
- U1 pad 91: /RD4r -> /RD4
- U1 pad 92: /RD5r -> /RD5
- U1 pad 95: /RD6r -> /RD6
- U1 pad 96: /RD0r -> /RD0
- U1 pad 97: /RD7r -> /RD7
- U1 pad 99: /RD2r -> /RD2
- U3 pad 11: Net-(RN5-Pad4) -> /Ain3
- U3 pad 12: Net-(RN5-Pad3) -> /Ain4
- U3 pad 13: Net-(RN5-Pad2) -> /Ain2
- U3 pad 14: Net-(RN5-Pad1) -> /Ain0
- U3 pad 15: Net-(RN4-Pad4) -> /Ain1
- U3 pad 16: Net-(RN4-Pad3) -> /Ain7
- U3 pad 17: Net-(RN4-Pad2) -> /~C07X~in
- U3 pad 18: Net-(RN4-Pad1) -> /R~W~in
Routing:
- net /RD5r: track 14.8 -> 0.00 mm, vias 2 -> 0
- net /RD5: track 20.3 -> 34.4 mm
- net /RD4r: track 14.0 -> 0.00 mm, vias 2 -> 0
- net /RD4: track 20.0 -> 33.2 mm
- net /RD3: track 19.5 -> 32.3 mm
- net /RD3r: track 12.7 -> 0.00 mm, vias 2 -> 0
- net /RD1r: track 12.6 -> 0.00 mm, vias 2 -> 0
- net /RD7: track 20.8 -> 32.7 mm
- net /RD1: track 19.3 -> 30.9 mm
- net /RD6: track 20.2 -> 31.5 mm
- net /RD7r: track 11.1 -> 0.00 mm, vias 2 -> 0
- net /RD6r: track 11.0 -> 0.00 mm, vias 2 -> 0
- net Net-(R4-Pad2): track 12.5 -> 3.31 mm
- net /RD0r: track 9.07 -> 0.00 mm, vias 2 -> 0
- net /RD0: track 18.6 -> 27.4 mm
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
Commit message: Generated gerbers and documentation
Parts:
- added D1: White, stdpads:LED_0805, F.Cu at (229.5, 98.8)
- added R8: 180, stdpads:R_0805, F.Cu at (229.5, 100.8)
- U1: value EPM240T100C5N -> EPM240T100
Connections:
- U1 pad 88: Net-(U1-Pad88) -> /LED
Routing:
- net /LED: track 0.00 -> 13.0 mm
- net +3V3: track 121.4 -> 128.0 mm, vias 78 -> 79
- net /TDI: track 89.0 -> 86.7 mm
- net Net-(D1-Pad2): track 0.00 -> 1.96 mm
- net /TDO: track 107.9 -> 107.3 mm
- net /TCK: track 85.7 -> 85.1 mm
- net GND: track 158.9 -> 159.4 mm, vias 286 -> 287
Other:
- board text added: "B20A"
