File: Hardware/MAX/RAM2E.kicad_pcb (KiCad board)
At the start: 4 copper layers, 78.2 x 50 mm, 76 parts, among them J1 AppleIIeAux, J2 microUSB, J3 C14M, J4 C14M, J5 JTAG, U1 5M240ZT100C5N, U10 CH340G, U11 74AHCT1G125GW, U2 W9812G6KH-6, U3 74AHC245PW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

Commit message: RC
Fix board IDs
Connections:
- U10 pad 11: +3V3 -> GND
- U10 pad 12: GND -> +3V3
Changed lines of the file:
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@@
       (net 60 "+3V3") (pinfunction "~{DSR}") (pintype "input"))
     (pad "11" smd roundrect (at 1.905 -2.475 180) (size 1.95 0.6) (layers "F.Cu" "F.Paste" "F.Mask") (roundrect_rratio 0.25)
-      (net 60 "+3V3") (pinfunction "~{RI}") (pintype "input"))
+      (net 2 "GND") (pinfunction "~{RI}") (pintype "input"))
     (pad "12" smd roundrect (at 0.635 -2.475 180) (size 1.95 0.6) (layers "F.Cu" "F.Paste" "F.Mask") (roundrect_rratio 0.25)
-      (net 2 "GND") (pinfunction "~{DCD}") (pintype "input"))
+      (net 60 "+3V3") (pinfunction "~{DCD}") (pintype "input"))
     (pad "13" smd roundrect (at -0.635 -2.475 180) (size 1.95 0.6) (layers "F.Cu" "F.Paste" "F.Mask") (roundrect_rratio 0.25)
       (net 61 "/TDI") (pinfunction "~{DTR}") (pintype "output"))
@@
   (segment (start 237.55 118.75) (end 237.35 118.95) (width 0.5) (layer "F.Cu") (net 2))
   (segment (start 226.6 106) (end 226.6 105.35) (width 0.508) (layer "F.Cu") (net 2))
+  (segment (start 200.979 111.5695) (end 199.5805 111.5695) (width 0.5) (layer "F.Cu") (net 2))
   (segment (start 237.05 116.0125) (end 237.05 114.9) (width 0.3) (layer "F.Cu") (net 2))
   (segment (start 266.6 109.85) (end 267.7 109.85) (width 0.5) (layer "F.Cu") (net 2))
@@
   (segment (start 261.2 104.4) (end 259.85 104.4) (width 1) (layer "F.Cu") (net 2))
   (segment (start 216.35 123.15) (end 215.65 123.15) (width 0.5) (layer "F.Cu") (net 2))
-  (segment (start 200.979 112.8395) (end 202.3745 112.8395) (width 0.5) (layer "F.Cu") (net 2))
   (segment (start 229.75 116.25) (end 229.75 115.35) (width 0.5) (layer "F.Cu") (net 2))
   (segment (start 215.65 123.15) (end 215.5 123) (width 0.5) (layer "F.Cu") (net 2))
@@
   (segment (start 210.3 106.8) (end 210.3 107.6) (width 0.5) (layer "F.Cu") (net 2))
   (segment (start 212.95 123.15) (end 213.1 123) (width 0.4) (layer "F.Cu") (net 2))
+  (segment (start 200.979 111.5695) (end 202.3745 111.5695) (width 0.5) (layer "F.Cu") (net 2))
   (segment (start 260.5 127.55) (end 260.5 128.7) (width 0.45) (layer "F.Cu") (net 2))
   (segment (start 235.475 123.15) (end 235.625 123.3) (width 0.508) (layer "F.Cu") (net 2))
   (segment (start 242.1 127.55) (end 242.75 127.55) (width 0.45) (layer "F.Cu") (net 2))
   (segment (start 244.55 100.6875) (end 244.55 101.7) (width 0.3) (layer "F.Cu") (net 2))
-  (segment (start 200.979 112.8395) (end 199.5805 112.8395) (width 0.5) (layer "F.Cu") (net 2))
   (segment (start 227.3 100.55) (end 226.6 100.55) (width 0.5) (layer "F.Cu") (net 2))
   (segment (start 213.55 123) (end 213.1 123) (width 0.4) (layer "F.Cu") (net 2))
@@
   (via (at 202.3745 116.459) (size 0.5) (drill 0.3) (layers "F.Cu" "B.Cu") (net 2))
   (via (at 199.8 103.5) (size 0.5) (drill 0.3) (layers "F.Cu" "B.Cu") (net 2))
+  (via (at 202.3745 111.5695) (size 0.5) (drill 0.3) (layers "F.Cu" "B.Cu") (net 2))
   (via (at 261.15 127.55) (size 0.5) (drill 0.3) (layers "F.Cu" "B.Cu") (net 2))
   (via (at 219.71 131.191) (size 0.5) (drill 0.3) (layers "F.Cu" "B.Cu") (net 2))
@@
   (via (at 226.6 101.4) (size 0.5) (drill 0.3) (layers "F.Cu" "B.Cu") (net 2))
   (via (at 250.19 92.964) (size 0.5) (drill 0.3) (layers "F.Cu" "B.Cu") (net 2))
+  (via (at 199.5805 111.5695) (size 0.5) (drill 0.3) (layers "F.Cu" "B.Cu") (net 2))
   (via (at 231.25 107.25) (size 0.5) (drill 0.3) (layers "F.Cu" "B.Cu") (net 2))
   (via (at 210.4 107.7) (size 0.5) (drill 0.3) (layers "F.Cu" "B.Cu") (net 2))
@@
   (via (at 265.2 104.4) (size 1) (drill 0.5) (layers "F.Cu" "B.Cu") (net 2))
   (via (at 210.15 100.1) (size 0.5) (drill 0.3) (layers "F.Cu" "B.Cu") (net 2))
-  (via (at 202.3745 112.8395) (size 0.5) (drill 0.3) (layers "F.Cu" "B.Cu") (net 2))
   (via (at 211.5 108.8) (size 0.5) (drill 0.3) (layers "F.Cu" "B.Cu") (net 2))
   (via (at 249.3 112.2) (size 0.5) (drill 0.3) (layers "F.Cu" "B.Cu") (net 2))
@@
   (via (at 229.75 115.35) (size 0.5) (drill 0.3) (layers "F.Cu" "B.Cu") (net 2))
   (via (at 232.4 101.55) (size 0.5) (drill 0.3) (layers "F.Cu" "B.Cu") (net 2))
-  (via (at 199.5805 112.8395) (size 0.5) (drill 0.3) (layers "F.Cu" "B.Cu") (net 2))
   (via (at 269.05 127.35) (size 0.5) (drill 0.3) (layers "F.Cu" "B.Cu") (net 2))
   (via (at 210.15 104.1) (size 0.5) (drill 0.3) (layers "F.Cu" "B.Cu") (net 2))
@@
   (segment (start 265.35 111.75) (end 265.25 111.65) (width 0.8) (layer "F.Cu") (net 60))
   (segment (start 226.75 98.1) (end 226.75 97.35) (width 0.5) (layer "F.Cu") (net 60))
-  (segment (start 200.979 111.5695) (end 199.5805 111.5695) (width 0.5) (layer "F.Cu") (net 60))
   (segment (start 244.05 100.6875) (end 244.05 101.7) (width 0.3) (layer "F.Cu") (net 60))
   (segment (start 213.05 93.15) (end 213.05 92.45) (width 0.5) (layer "F.Cu") (net 60))
@@
   (segment (start 214.15 115.85) (end 214.2 115.8) (width 0.45) (layer "F.Cu") (net 60))
   (segment (start 258.5 108) (end 258.5 109.1) (width 0.8) (layer "F.Cu") (net 60))
+  (segment (start 200.979 112.8395) (end 202.3745 112.8395) (width 0.5) (layer "F.Cu") (net 60))
   (segment (start 243.05 117.2) (end 243.4 117.2) (width 0.5) (layer "F.Cu") (net 60))
   (segment (start 237.05 100.675) (end 237.05 101.8) (width 0.3) (layer "F.Cu") (net 60))
@@
   (segment (start 213.05 117.95) (end 213.05 116.55) (width 0.8) (layer "F.Cu") (net 60))
   (segment (start 243.55 116.0125) (end 243.55 117.05) (width 0.4) (layer "F.Cu") (net 60))
-  (segment (start 200.979 111.5695) (end 202.3745 111.5695) (width 0.5) (layer "F.Cu") (net 60))
   (segment (start 226.6 98.25) (end 226.6 99.05) (width 0.5) (layer "F.Cu") (net 60))
+  (segment (start 200.979 112.8395) (end 199.5805 112.8395) (width 0.5) (layer "F.Cu") (net 60))
   (segment (start 213.05 115.85) (end 213.05 116.55) (width 0.45) (layer "F.Cu") (net 60))
   (segment (start 248.75 110.35) (end 247.7125 110.35) (width 0.3) (layer "F.Cu") (net 60))
@@
   (via (at 235.2 117.95) (size 0.5) (drill 0.3) (layers "F.Cu" "B.Cu") (net 60))
   (via (at 226.25 127.55) (size 0.5) (drill 0.3) (layers "F.Cu" "B.Cu") (net 60))
-  (via (at 202.3745 111.5695) (size 0.5) (drill 0.3) (layers "F.Cu" "B.Cu") (net 60))
   (via (at 236.7 97.8) (size 0.5) (drill 0.3) (layers "F.Cu" "B.Cu") (net 60))
   (via (at 236.9 99.5) (size 0.5) (drill 0.3) (layers "F.Cu" "B.Cu") (net 60))
@@
   (via (at 204.5335 114.1095) (size 0.5) (drill 0.3) (layers "F.Cu" "B.Cu") (net 60))
   (via (at 207.3275 114.3) (size 0.5) (drill 0.3) (layers "F.Cu" "B.Cu") (net 60))
-  (via (at 199.5805 111.5695) (size 0.5) (drill 0.3) (layers "F.Cu" "B.Cu") (net 60))
   (via (at 199.5805 117.9195) (size 0.5) (drill 0.3) (layers "F.Cu" "B.Cu") (net 60))
   (via (at 223.05 94.05) (size 0.5) (drill 0.3) (layers "F.Cu" "B.Cu") (net 60))
@@
   (via (at 223.05 117.1) (size 0.5) (drill 0.3) (layers "F.Cu" "B.Cu") (net 60))
   (via (at 251.05 110.7) (size 0.5) (drill 0.3) (layers "F.Cu" "B.Cu") (net 60))
+  (via (at 202.3745 112.8395) (size 0.5) (drill 0.3) (layers "F.Cu" "B.Cu") (net 60))
   (via (at 199.5805 110.2995) (size 0.5) (drill 0.3) (layers "F.Cu" "B.Cu") (net 60))
   (via (at 232.1 116.25) (size 0.5) (drill 0.3) (layers "F.Cu" "B.Cu") (net 60))
@@
   (via (at 243.05 118.9) (size 0.5) (drill 0.3) (layers "F.Cu" "B.Cu") (net 60))
   (via (at 258.5 109.1) (size 1) (drill 0.5) (layers "F.Cu" "B.Cu") (net 60))
+  (via (at 199.5805 112.8395) (size 0.5) (drill 0.3) (layers "F.Cu" "B.Cu") (net 60))
   (via (at 266.6 112.8) (size 1) (drill 0.5) (layers "F.Cu" "B.Cu") (net 60))
   (via (at 200.5965 118.618) (size 0.5) (drill 0.3) (layers "F.Cu" "B.Cu") (net 60))

Commit message: RC
Parts:
- added R11: 10k, stdpads:R_0603, F.Cu at (257.2, 112.0)
- added R12: 10k, stdpads:R_0603, F.Cu at (257.2, 115.2)
Routing:
- net /V~{OE}: track 5.99 -> 20.6 mm, vias 0 -> 2
- net /D~{OE}: track 16.3 -> 22.2 mm, vias 2 -> 3
- net +3V3: track 141.5 -> 143.0 mm, vias 87 -> 88
- net GND: vias 281 -> 279

Commit message: RC
Parts:
- U3, U5: value 74AHC245PW -> 74LVC245APW
Other:
- board text added: "C10A"
- board text removed: "B21A"
