File: Hardware/MAX/RAM2E.sch (KiCad schematic (older format))
At the start: 62 parts, among them J1 AppleIIeAux, J2 JTAG, J3 C14M, U1 EPM240T100C5N, U2 W9812G6KH-6, U3 74LVC245APW, U4 74LVC245APW, U5 74LVC245APW, U6 74AHCT245PW, U7 74AHCT245PW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

Commit message: still workin
Connections:
- net RD0r: now also RN1.8 (R1.2), U1.96 (IO2_96); no longer RN2.5 (R4.2), U1.97 (IO2_97)
- net RD7r: now also RN2.5 (R4.2), U1.97 (IO2_97); no longer RN1.8 (R1.2), U1.96 (IO2_96)
Changed lines of the file:
@@
 	6900 5450 7100 5450
 Wire Wire Line
-	7100 5250 6900 5250
+	7100 6050 6900 6050
 Wire Wire Line
 	7100 5350 6900 5350
@@
 Wire Wire Line
 	3600 3250 3400 3250
-Text Label 6900 5250 0    50   ~ 0
+Text Label 6900 6050 0    50   ~ 0
 RD7r
 Text Label 6900 5350 0    50   ~ 0
@@
 Text Label 6900 5750 0    50   ~ 0
 RD4r
-Text Label 6900 6050 0    50   ~ 0
+Text Label 6900 5250 0    50   ~ 0
 RD0r
 Text Label 6900 5950 0    50   ~ 0
@@
 RD5r
 Wire Wire Line
-	7100 6050 6900 6050
+	7100 5250 6900 5250
 Wire Wire Line
 	7100 5950 6900 5950
@@
 Text Label 6800 5950 2    50   ~ 0
 RD2r
+Text Label 6800 5650 2    50   ~ 0
+RD0r
 Text Label 6800 5750 2    50   ~ 0
-RD0r
-Text Label 6800 5650 2    50   ~ 0
 RD7r
 Text Label 6800 5550 2    50   ~ 0
@@
 RD5r
 Wire Wire Line
+	6600 5650 6800 5650
+Wire Wire Line
 	6600 5750 6800 5750
-Wire Wire Line
-	6600 5650 6800 5650
 Wire Wire Line
 	6600 5550 6800 5550
@@
 	-1   0    0    -1
 $EndComp
-Wire Bus Line
-	8200 4250 8200 5350
-$Comp
-L power:+1V8 #PWR?
+$Comp
+L power:+1V8 #PWR0136
 U 1 1 60997BFF
 P 8600 750
-F 0 "#PWR?" H 8600 600 50  0001 C CNN
+F 0 "#PWR0136" H 8600 600 50  0001 C CNN
 F 1 "+1V8" H 8600 900 50  0000 C CNN
 F 2 "" H 8600 750 50  0001 C CNN
@@
 	1    0    0    -1
 $EndComp
+Wire Bus Line
+	8200 4250 8200 5350
 $EndSCHEMATC

Commit message: idk
Parts:
- removed RN1, RN2, RN3, RN4, RN5: 4x33, stdpads:R4_0402, symbol Device:R_Pack04
- added R4, R5: 47, stdpads:R_0603, symbol Device:R_Small
Connections:
- net RD0r is gone; now on net RD0: U1.96 (IO2_96)
- net RD1r is gone; now on net RD1: U1.90 (IO2_90)
- net RD2r is gone; now on net RD2: U1.99 (IO2_99)
- net RD3r is gone; now on net RD3: U1.89 (IO2_89)
- net RD4r is gone; now on net RD4: U1.91 (IO2_91)
- net RD5r is gone; now on net RD5: U1.92 (IO2_92)
- net RD6r is gone; now on net RD6: U1.95 (IO2_95)
- net RD7r is gone; now on net RD7: U1.97 (IO2_97)
- net ACLK: now also R5.1
- net Ain0: now also U3.14 (B4)
- net Ain1: now also U3.15 (B3)
- net Ain2: now also U3.13 (B5)
- net Ain3: now also U3.11 (B7)
- net Ain4: now also U3.12 (B6)
- net Ain7: now also U3.16 (B2)
- net RCLK: now also R4.1
- net R~W~in: now also U3.18 (B0)
- net ~C07X~in: now also U3.17 (B1)
- net at U4.18 (B0): now also R4.2, R5.2
- no-connect marks 17 -> 13
Other:
- moved on the sheet: R3

Commit message: Generated gerbers and documentation
Parts:
- added D1: White, stdpads:LED_0805, symbol Device:LED_Small_ALT
- added R8: 180, stdpads:R_0805, symbol Device:R_Small
- R1, R6: Mfg. Part Numbers Uniroyal 0805W8F2202T5E -> Uniroyal 0805W8F0000T5E
- U1: value EPM240T100C5N -> EPM240T100
- U2: Notes Most 166 MHz 128/256 Mbit SDRAM is acceptable. -> Most 166 MHz 128/256 Mbit x16 SDRAM is acceptable.
- U3, U4, U5: Mfg. Part Numbers NXP 74LVC245APW, TI SN74LVC245APW -> NXP 74LVC245APW, TI SN74LVC245APW, NXP 74AHC245PW, NXP 74AH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; Notes (none) -> Most 74LVC245 or 74AHC245 in TSSOP-20 package is acceptable.
- U6, U7: Mfg. Part Numbers NXP 74AHCT245PW, TI SN74AHCT245PW -> NXP 74AHCT245PW, NXP 74AHCT245APW, TI SN74AHCT245PW; Notes (none) -> Most 74AHCT245 in TSSOP-20 package is acceptable.
- U8: Notes (none) -> Most 3.3V regulator in SOT-23 package is acceptable.
- U9: LCSC Part (none) -> C151375; Notes (none) -> Most 1.8V regulator in SOT-23-5 package is acceptable.
Connections:
- net +3V3: now also R8.2
- net LED: now reaches U1.88 (IO2_88)
- net LED: now also D1.1 (K)
- new net: D1.2 (A), R8.1
- no-connect marks 13 -> 12

Commit message: BOM finished
Parts:
- U1: Mfg. Part Numbers Altera 5M240ZT100C5N , Altera 5M240ZT100C4N, Altera 5M240ZT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 -> Altera 5M240ZT100C5N, Altera 5M240ZT100C4N, Altera 5M240ZT1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
Changed lines of the file:
@@
 F 3 "" H 5600 4050 50  0001 C CNN
 F 4 "C10041" H 5600 4050 50  0001 C CNN "LCSC Part"
-F 5 "Altera 5M240ZT100C5N , Altera 5M240ZT100C4N, Altera 5M240ZT100C3N, Altera 5M240ZT100I5N, Altera 5M240ZT100I4N, Altera 5M240ZT100A5N, Altera 5M240ZT100A4N, Altera EPM240T100C5N, Altera EPM240T100C4N, Altera EPM240T100C3N, Altera EPM240T100I5N, Altera EPM240T100I4N, Altera EPM240T100A5N, Altera EPM240T100A4N, AGM/Alta-Gate AG256SL100, AGM AG256SL100C3, AGM AG256SL100C4, AGM/Alta-Gate AG272SL100, AGM AG272SL100C3, AGM AG272SL100C4, AGM/Alta-Gate AG576SL100, AGM AG576SL100C3, AGM AG576SL100C4" H 5600 4050 50  0001 C CNN "Mfg. Part Numbers"
+F 5 "Altera 5M240ZT100C5N, Altera 5M240ZT100C4N, Altera 5M240ZT100C3N, Altera 5M240ZT100I5N, Altera 5M240ZT100I4N, Altera 5M240ZT100A5N, Altera 5M240ZT100A4N, Altera EPM240T100C5N, Altera EPM240T100C4N, Altera EPM240T100C3N, Altera EPM240T100I5N, Altera EPM240T100I4N, Altera EPM240T100A5N, Altera EPM240T100A4N, AGM/Alta-Gate AG256SL100, AGM AG256SL100C3, AGM AG256SL100C4, AGM/Alta-Gate AG272SL100, AGM AG272SL100C3, AGM AG272SL100C4, AGM/Alta-Gate AG576SL100, AGM AG576SL100C3, AGM AG576SL100C4" H 5600 4050 50  0001 C CNN "Mfg. Part Numbers"
 	1    5600 4050
 	1    0    0    -1
