File: Hardware/MAX/Docs.kicad_sch (KiCad schematic)
At the start: 0 parts

Commit message: As sent to testers
Other:
- note added: "PCall"
- note added: "RD"
- note added: "WR"
- note removed: "RD+AP"
- note removed: "WR+AP"
