File: Hardware/MAX/Docs.kicad_sch (KiCad schematic)
At the start: 0 parts

Commit message: RC
Other:
- title: GW4203B (RAM2E II) - EPM240 / 5M240Z / AG256 -> GW4203C (RAM2E II) - EPM240 / 5M240Z / AG256
Changed lines of the file:
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@@
   (paper "A4")
   (title_block
-    (title "GW4203B (RAM2E II) - EPM240 / 5M240Z / AG256")
-    (date "2024-04-24")
-    (rev "2.1")
+    (title "GW4203C (RAM2E II) - EPM240 / 5M240Z / AG256")
+    (date "2024-05-20")
+    (rev "1.0")
     (company "Garrett's Workshop")
   )
