File: Hardware/MAX/RAM2E.kicad_sch (KiCad schematic)
At the start: 76 parts, among them J1 AppleIIeAux, J2 microUSB, J3 C14M, J4 C14M, J5 JTAG, U1 5M240ZT100C5N, U10 CH340G, U11 74AHCT1G125GW, U2 W9812G6KH-6, U3 74LVC245APW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

Commit message: RC C.1.1
Parts:
- H1, H2, H3, H4, H5: value (none) -> (none)
- R1: value 0 -> 0
Connections:
- no-connect marks 12 -> 13
