File: Hardware/LCMXO/RAM2E.kicad_pcb (KiCad board)
At the start: 4 copper layers, 78.2 x 50 mm, 66 parts, among them J1 AppleIIeAux, J2 JTAG, J3 C14M, U1 LCMXO256-TQFP-100, U2 W9812G6KH-6, U3 74LVC245APW, U4 74LVC245APW, U5 74LVC245APW, U6 74AHCT245PW, U7 74AHCT245PW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

Commit message: still workin
Parts:
- removed the C11 at (230.3, 107.3)
- removed the C29 at (246.3, 118.0)
- removed the C9 at (239.1, 118.0)
- removed R10: 22k, stdpads:R_0805
- removed REF**: SOIC-8_3.9mm, stdpads:SOIC-8_3.9mm
- removed RN1, RN2, RN3, RN4, RN5: 4x33, stdpads:R4_0402
- added C30: 2u2, stdpads:C_0603, F.Cu at (273.9, 99.2)
- added C31: 2u2, stdpads:C_0603, F.Cu at (205.5, 106.3)
- added R4: 47, stdpads:R_0603, F.Cu at (226.8, 119.0)
- added R5: 47, stdpads:R_0603, F.Cu at (228.2, 119.0)
- added R8: 47, stdpads:R_0603, F.Cu at (205.5, 109.2)
- added U11: 25F010, stdpads:SOIC-8_5.3mm, F.Cu at (268.0, 100.3)
- R9: value 22k -> 10k; footprint stdpads:R_0805 -> stdpads:R_0603
- U1: value LCMXO256-TQFP-100 -> LCMXO640-3TN100C
- U9: value AP2127K-1.8TRG1 -> AP2127K-1.2TRG1
- moved C18 43.8 mm to (241.1, 98.7), turned to 180 degrees
- moved C19 41.9 mm to (249.7, 110.6), turned to 270 degrees
- moved C17 37.0 mm to (249.7, 107.1), turned to 270 degrees
- moved C16 19.6 mm to (230.3, 110.2)
- moved C15 17.8 mm to (246.3, 118.0), turned to 0 degrees
- moved C13 13.8 mm to (230.3, 107.3), turned to 90 degrees
- moved C14 13.0 mm to (239.1, 118.0), turned to 0 degrees
- moved C25 2.05 mm to (223.8, 118.0), turned to 0 degrees
- moved R9 1.82 mm to (205.5, 107.8)
Connections:
- C16 pad 1: +3V3 -> +1V2
- C19 pad 1: +1V8 -> +1V2
- C4 pad 1: +1V8 -> +1V2
- C5 pad 1: +1V8 -> +1V2
- J2 pad 10: GND -> Net-(J2-Pad10)
- J2 pad 3: /TDO -> /TMS
- J2 pad 4: +3V3 -> GND
- J2 pad 5: /TMS -> /TDI
- J2 pad 6: Net-(J2-Pad6) -> +3V3
- J2 pad 7: Net-(J2-Pad7) -> /TDO
- J2 pad 9: /TDI -> Net-(J2-Pad9)
- R1 pad 2: +1V8 -> +1V2
- R9 pad 1: /TCK -> /TCKr
- U1 pad 100: /~WE~ -> /RA7
- U1 pad 11: /Ain1 -> /Ain2
- U1 pad 13: /Ain7 -> /Ain3
- U1 pad 2: /Ain2 -> /Ain7
- U1 pad 27: Net-(U1-Pad27) -> /V~OE~
- U1 pad 29: Net-(U1-Pad29) -> +3V3
- U1 pad 30: Net-(U1-Pad30) -> GND
- U1 pad 32: Net-(U1-Pad32) -> /Vout7
- U1 pad 33: /TCK -> /TCKr
- U1 pad 34: Net-(U1-Pad34) -> /Vout3
- U1 pad 36: Net-(U1-Pad36) -> /Vout6
- U1 pad 37: Net-(U1-Pad37) -> /Vout1
- U1 pad 38: Net-(U1-Pad38) -> /Vout5
- U1 pad 39: Net-(U1-Pad39) -> /Vout4
- U1 pad 4: /Ain4 -> /Ain0
- U1 pad 43: Net-(U1-Pad43) -> /D~OE~
- U1 pad 44: Net-(U1-Pad44) -> /Dout5
- U1 pad 45: Net-(U1-Pad45) -> /Dout4
- U1 pad 46: Net-(U1-Pad46) -> /Dout2
- U1 pad 47: Net-(U1-Pad47) -> /Dout3
- U1 pad 48: GND -> +3V3
- U1 pad 49: Net-(U1-Pad49) -> /Dout1
- U1 pad 50: Net-(U1-Pad50) -> /Dout0
- U1 pad 51: Net-(U1-Pad51) -> /Dout6
- U1 pad 52: Net-(U1-Pad52) -> /Dout7
- U1 pad 53: Net-(U1-Pad53) -> /MOSI
- U1 pad 54: Net-(U1-Pad54) -> /SCK
- U1 pad 55: Net-(U1-Pad55) -> /Vout0
- U1 pad 56: Net-(U1-Pad56) -> /MISO
- U1 pad 57: Net-(U1-Pad57) -> /Vout2
- U1 pad 58: Net-(U1-Pad58) -> /S~CS~
- U1 pad 6: /Ain3 -> /Ain4
- U1 pad 61: Net-(U1-Pad61) -> /DQML
- U1 pad 63: Net-(U1-Pad63) -> /BA0
- U1 pad 64: Net-(U1-Pad64) -> /RD0
- U1 pad 65: Net-(U1-Pad65) -> /RD1
- U1 pad 66: Net-(U1-Pad66) -> /RD2
- U1 pad 67: Net-(U1-Pad67) -> /RD3
- U1 pad 68: Net-(U1-Pad68) -> /RD4
- U1 pad 69: Net-(U1-Pad69) -> /RD5
- U1 pad 70: Net-(U1-Pad70) -> /RD6
- U1 pad 71: Net-(U1-Pad71) -> /RD7
- U1 pad 72: /DQMH -> /~CAS~
- U1 pad 73: /DQML -> /~RAS~
- U1 pad 76: /RA4 -> /DQMH
- U1 pad 77: /RA6 -> /~CS~
- U1 pad 78: /RA1 -> /~WE~
- U1 pad 79: /RA7 -> /RA11
- U1 pad 80: /RA0 -> +3V3
- U1 pad 81: /RA8 -> GND
- U1 pad 82: /RA10 -> /CKE
- U1 pad 83: /RA9 -> /BA1
- U1 pad 85: /BA1 -> /RA9
- U1 pad 87: /RA3 -> /RA10
- U1 pad 89: /RA2 -> /RA1
- U1 pad 9: /Ain0 -> /Ain1
- U1 pad 91: /RA5 -> /RA6
- U1 pad 94: /~CS~ -> /RA2
- U1 pad 95: /RA11 -> /RA5
- U1 pad 96: /BA0 -> /RA8
- U1 pad 97: /~RAS~ -> /RA3
- U1 pad 98: /CKE -> /RA0
- U1 pad 99: /~CAS~ -> /RA4
- U3 pad 11: Net-(RN5-Pad4) -> /Ain3
- U3 pad 12: Net-(RN5-Pad3) -> /Ain4
- U3 pad 13: Net-(RN5-Pad2) -> /Ain2
- U3 pad 14: Net-(RN5-Pad1) -> /Ain0
- U3 pad 15: Net-(RN4-Pad4) -> /Ain1
- U3 pad 16: Net-(RN4-Pad3) -> /Ain7
- U3 pad 17: Net-(RN4-Pad2) -> /~C07X~in
- U3 pad 18: Net-(RN4-Pad1) -> /R~W~in
- U9 pad 5: +1V8 -> +1V2
Routing:
- net +1V2: track 33.1 -> 107.5 mm, vias 3 -> 9
- net /TCKr: track 0.00 -> 73.8 mm, vias 0 -> 2
- net /TCK: track 61.1 -> 4.13 mm, vias 2 -> 0
- net +1V8: track 38.3 -> 0.00 mm, vias 6 -> 0
- net /SCK: track 0.00 -> 31.1 mm
- net /MOSI: track 0.00 -> 30.1 mm
- net /Dout7: track 0.95 -> 30.5 mm
- net /Vout2: track 0.95 -> 29.2 mm, vias 0 -> 2
- net /Vout0: track 0.95 -> 28.4 mm, vias 0 -> 2
- net /Dout6: track 1.15 -> 28.0 mm
- net /S~CS~: track 0.00 -> 25.3 mm
- net /MISO: track 0.00 -> 24.3 mm
- net /Dout0: track 1.35 -> 25.2 mm
- net /Dout1: track 1.55 -> 24.4 mm
- net /Vout4: track 0.95 -> 23.3 mm, vias 0 -> 2
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- added copper zone on F.Cu, net +1V2
- removed copper zone on F.Cu, net +1V8

Commit message: Generated gerbers and documentation
Parts:
- added D1: White, stdpads:LED_0805, F.Cu at (229.5, 98.8)
- added R10: 180, stdpads:R_0805, F.Cu at (229.5, 100.8)
- C31: value 2u2 -> 15p
- U1: value LCMXO640-3TN100C -> LCMXO256-TN100
Connections:
- U1 pad 59: Net-(U1-Pad59) -> /LED
Routing:
- net /LED: track 0.00 -> 17.4 mm
- net +3V3: track 135.2 -> 140.0 mm, vias 89 -> 90
- net Net-(D1-Pad2): track 0.00 -> 1.96 mm
- net /TDO: track 84.9 -> 85.7 mm
- net /DQMH: track 10.0 -> 10.8 mm
- net /TCKr: track 73.8 -> 73.2 mm
- net GND: vias 272 -> 271
Other:
- board text added: "B20B"
