File: Hardware/LCMXO/RAM2E.sch (KiCad schematic (older format))
At the start: 62 parts, among them J1 AppleIIeAux, J2 JTAG, J3 C14M, U1 EPM240T100C5N, U2 W9812G6KH-6, U3 74LVC245APW, U4 74LVC245APW, U5 74LVC245APW, U6 74AHCT245PW, U7 74AHCT245PW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

Commit message: started
Parts:
- removed U1: EPM240T100C5N, stdpads:TQFP-100_14x14mm_P0.5mm, symbol GW_PLD:5M240ZT100
- added U1: LCMXO256-TQFP-100, stdpads:TQFP-100, symbol GW_PLD:LCMXO256-TQFP-100
- C1, C2, C29, C3, C4, C5, C6: Mfg. Part Numbers (none) -> Samsung CL21A106KAYNNNE; Notes (none) -> 10V or higher. Any manufacturer's part is acceptable but Sa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
- C10, C11, C12, C13, C14, C15, C16, C17, C18, C19, C20, C21, C22, C23, C24, C25, C26, C27, C28, C7, C8, C9: Mfg. Part Numbers (none) -> Samsung CL10A225KO8NNNC; Notes (none) -> 10V or higher. Any manufacturer's part is acceptable but Sa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
- FID1, FID2, FID3, FID4: Notes (none) -> DNP - SMT vision system fiducial
- H1, H2, H3, H4: Notes (none) -> DNP - mounting hole for solder paste printing
- H5: Notes (none) -> DNP - mounting hole
- J1: Notes (none) -> DNP - edge connector
- J2: Notes (none) -> DNP - test pad connector
- J3: Notes (none) -> DNP
- R1: value 0 -> 0; Mfg. Part Numbers (none) -> Uniroyal 0805W8F2202T5E; Notes (none) -> Any manufacturer's part is acceptable.
- R10, R6, R9: Mfg. Part Numbers (none) -> Uniroyal 0805W8F2202T5E; Notes (none) -> Any manufacturer's part is acceptable.
- R2, R3: Mfg. Part Numbers (none) -> Uniroyal 0603WAF470JT5E; Notes (none) -> Any manufacturer's part is acceptable.
- RN1, RN2, RN3, RN4, RN5: Mfg. Part Numbers (none) -> Uniroyal 4D02WGJ0330TCE; Notes (none) -> Any manufacturer's part is acceptable.
- U2: Mfg. Part Numbers (none) -> Winbond W9812G6KH-6, Winbond W9812G6KH-6I, Winbond W9825G6K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; Notes (none) -> Most 166 MHz 128/256 Mbit SDRAM is acceptable.
- U3, U4, U5: Mfg. Part Numbers (none) -> NXP 74LVC245APW, TI SN74LVC245APW
- U6, U7: Mfg. Part Numbers (none) -> NXP 74AHCT245PW, TI SN74AHCT245PW
- U8: Mfg. Part Numbers (none) -> Torex XC6206P332MR
- U9: value DNP -> AP2127K-1.2TRG1; symbol Regulator_Linear:AP2127K-1.8 -> Regulator_Linear:AP2127K-1.2
Connections:
- net labels added: +1V2
- net labels removed: +1V8
- wire segments 276 -> 277
- no-connect marks 17 -> 15

Commit message: still workin
Parts:
- removed R10: 22k, stdpads:R_0805, symbol Device:R_Small
- removed RN1, RN2, RN3, RN4, RN5: 4x33, stdpads:R4_0402, symbol Device:R_Pack04
- removed U1: LCMXO256-TQFP-100, stdpads:TQFP-100, symbol GW_PLD:LCMXO256-TQFP-100
- added C30, C31: 2u2, stdpads:C_0603, symbol Device:C_Small
- added R4, R5, R8: 47, stdpads:R_0603, symbol Device:R_Small
- added U1: LCMXO640-3TN100C, stdpads:TQFP-100_14x14mm_P0.5mm, symbol GW_PLD:LCMXO640-TQFP-100
- added U11: 25F010, stdpads:SOIC-8_5.3mm, symbol GW_RAM:SPIFlash-SO-8
- R9: value 22k -> 10k; footprint stdpads:R_0805 -> stdpads:R_0603
Connections:
- net labels added: MISO, MOSI, SCK, S~CS~, TCKr
- net labels removed: RD0r, RD1r, RD2r, RD3r, RD4r, RD5r, RD6r, RD7r, ~80VID~in
- wire segments 277 -> 265
- no-connect marks 15 -> 4
Other:
- moved on the sheet: C16, C19, R3

Commit message: Generated gerbers and documentation
Parts:
- added D1: White, stdpads:LED_0805, symbol Device:LED_Small_ALT
- added R10: 180, stdpads:R_0805, symbol Device:R_Small
- C31: value 2u2 -> 15p; LCSC Part C23630 -> (none); Mfg. Part Numbers Samsung CL10A225KO8NNNC -> (none)
- R1, R6: Mfg. Part Numbers Uniroyal 0805W8F2202T5E -> Uniroyal 0805W8F0000T5E
- R9: LCSC Part C17560 -> C25804; Mfg. Part Numbers Uniroyal 0805W8F2202T5E -> Uniroyal 0603WAF1002T5E
- U1: value LCMXO640-3TN100C -> LCMXO256-TN100; LCSC Part (none) -> C1550734; Mfg. Part Numbers (none) -> Lattice LCMXO256C-3TN100C, Lattice LCMXO256C-4TN100C, Latti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
- U11: LCSC Part (none) -> C2687406; Mfg. Part Numbers (none) -> Zetta ZD25WD20BTIGT, Adesto AT25SF081-SSHD, Winbond W25X20C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; Notes (none) -> Most SPI flash in SOIC-8 (3.9mm / 150 mil width) package is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
- U2: Notes Most 166 MHz 128/256 Mbit SDRAM is acceptable. -> Most 166 MHz 128/256 Mbit x16 SDRAM is acceptable.
- U3, U4, U5: Mfg. Part Numbers NXP 74LVC245APW, TI SN74LVC245APW -> NXP 74LVC245APW, TI SN74LVC245APW, NXP 74AHC245PW, NXP 74AH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; Notes (none) -> Most 74LVC245 or 74AHC245 in TSSOP-20 package is acceptable.
- U6, U7: Mfg. Part Numbers NXP 74AHCT245PW, TI SN74AHCT245PW -> NXP 74AHCT245PW, NXP 74AHCT245APW, TI SN74AHCT245PW; Notes (none) -> Most 74AHCT245 in TSSOP-20 package is acceptable.
- U8: Notes (none) -> Most 3.3V regulator in SOT-23 package is acceptable.
- U9: LCSC Part (none) -> C151376; Mfg. Part Numbers (none) -> Diodes AP2127K-1.2TRG1, Torex XC6228D122VR; Notes (none) -> Most 1.2V regulator in SOT-23-5 package is acceptable.
Connections:
- net +3V3: now also R10.2
- net LED: now reaches U1.59 (PR9D)
- net LED: now also D1.1 (K)
- new net: D1.2 (A), R10.1
- no-connect marks 4 -> 5
