File: Hardware/LCMXO2/RAM2E.sch (KiCad schematic (older format))
At the start: 62 parts, among them J1 AppleIIeAux, J2 JTAG, J3 C14M, U2 W9812G6KH-6, U3 74LVC245APW, U4 74LVC245APW, U5 74LVC245APW, U6 74AHCT245PW, U7 74AHCT245PW, U8 XC6206P332MR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

Commit message: still workin
Parts:
- removed R10: 22k, stdpads:R_0805, symbol Device:R_Small
- removed RN1, RN2, RN3, RN4, RN5: 4x33, stdpads:R4_0402, symbol Device:R_Pack04
- added C30, C31: 2u2, stdpads:C_0603, symbol Device:C_Small
- added R11, R5, R8: 10k, stdpads:R_0603, symbol Device:R_Small
- added R12, R13, R4: 47, stdpads:R_0603, symbol Device:R_Small
- R9: value 22k -> 10k; footprint stdpads:R_0805 -> stdpads:R_0603
- gave numbers to parts that had none: 1
Connections:
- net labels added: DONE, TCKr, ~INIT~, ~PROG~
- net labels removed: RD0r, RD1r, RD2r, RD3r, RD4r, RD5r, RD6r, RD7r, ~80VID~in
- wire segments 278 -> 268
- no-connect marks 15 -> 4
Other:
- moved on the sheet: C16, C19, R3

Commit message: Generated gerbers and documentation
Parts:
- added D1: White, stdpads:LED_0805, symbol Device:D_Small_ALT
- added R10: 180, stdpads:R_0805, symbol Device:R_Small
- C31: value 2u2 -> 15p; LCSC Part C23630 -> C1644; Mfg. Part Numbers Samsung CL10A225KO8NNNC -> Samsung CL10C150JB8NNNC
- R1, R6: Mfg. Part Numbers Uniroyal 0805W8F2202T5E -> Uniroyal 0805W8F0000T5E
- R11, R5, R8, R9: LCSC Part C17560 -> C25804; Mfg. Part Numbers Uniroyal 0805W8F2202T5E -> Uniroyal 0603WAF1002T5E
- U1: value LCMXO2-640-TG100 -> LCMXO2-TG100; footprint stdpads:TQFP-100 -> stdpads:TQFP-100_14x14mm_P0.5mm; LCSC Part (none) -> C1519051; Mfg. Part Numbers (none) -> Lattice LCMXO2-640HC-4TG100C, Lattice LCMXO2-640HC-5TG100C,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
- U2: Notes Most 166 MHz 128/256 Mbit SDRAM is acceptable. -> Most 166 MHz 128/256 Mbit x16 SDRAM is acceptable.
- U3, U4, U5: Mfg. Part Numbers NXP 74LVC245APW, TI SN74LVC245APW -> NXP 74LVC245APW, TI SN74LVC245APW, NXP 74AHC245PW, NXP 74AH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; Notes (none) -> Most 74LVC245 or 74AHC245 in TSSOP-20 package is acceptable.
- U6, U7: Mfg. Part Numbers NXP 74AHCT245PW, TI SN74AHCT245PW -> NXP 74AHCT245PW, NXP 74AHCT245APW, TI SN74AHCT245PW; Notes (none) -> Most 74AHCT245 in TSSOP-20 package is acceptable.
- U8: Notes (none) -> Most 3.3V regulator in SOT-23 package is acceptable.
- U9: LCSC Part (none) -> C151376; Mfg. Part Numbers (none) -> Diodes AP2127K-1.2TRG1, Torex XC6228D122VR; Notes (none) -> Most 1.2V regulator in SOT-23-5 package is acceptable.
Connections:
- net +3V3: now also R10.2
- net LED: now reaches U1.35 (PB6D/PCLKC_0)
- net LED: now also D1.1 (K)
- new net: D1.2 (A), R10.1
