File: Hardware/LCMXO2/RAM2E.kicad_pcb (KiCad board)
At the start: 4 copper layers, 78.2 x 50 mm, 66 parts, among them J1 AppleIIeAux, J2 JTAG, J3 C14M, U1 LCMXO2-TG100, U2 W9812G6KH-6, U3 74LVC245APW, U4 74LVC245APW, U5 74LVC245APW, U6 74AHCT245PW, U7 74AHCT245PW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

Commit message: 2.1?
Parts:
- added G***: LOGO, LOGO, F.Cu at (240.1, 93.4)
- added G***: LOGO, LOGO, F.Cu at (261.2, 93.3)
- D1: value White -> Amber
- R10: value 180 -> 220
- turned U2 to -90 degrees
- turned U9 to 90 degrees
Connections:
- net /D~OE~ renamed /D~{OE}
- net /R~W~ renamed /R~{W}
- net /R~W~80 renamed /R~{W}80
- net /R~W~80in renamed /R~{W}80in
- net /R~W~in renamed /R~{W}in
- net /V~OE~ renamed /V~{OE}
- net /~80VID~ renamed /~{80VID}
- net /~ALTVID~ renamed /~{ALTVID}
- net /~C07X~ renamed /~{C07X}
- net /~C07X~in renamed /~{C07X}in
- net /~CASEN~ renamed /~{CASEN}
- net /~CAS~ renamed /~{CAS}
- net /~CLRGAT~ renamed /~{CLRGAT}
- net /~CS~ renamed /~{CS}
- net /~EN80~ renamed /~{EN80}
- net /~EN80~in renamed /~{EN80}in
- net /~ENTMG~ renamed /~{ENTMG}
- net /~ENVID~ renamed /~{ENVID}
- net /~FRCTXT~ renamed /~{FRCTXT}
- net /~INIT~ renamed /~{INIT}
- net /~LDPS~ renamed /~{LDPS}
- net /~PCAS~ renamed /~{PCAS}
- net /~PRAS~ renamed /~{PRAS}
- net /~PROG~ renamed /~{PROG}
- net /~RA10~ renamed /~{RA10}
- net /~RA9~ renamed /~{RA9}
- net /~RAS~ renamed /~{RAS}
- net /~SEROUT~ renamed /~{SEROUT}
- net /~SYNC~ renamed /~{SYNC}
- net /~WE~ renamed /~{WE}
- net /~WNDW~ renamed /~{WNDW}
- J2 pad 10: Net-(J2-Pad10) -> unconnected-(J2-Pin_10-Pad10)
- J2 pad 8: Net-(J2-Pad8) -> unconnected-(J2-Pin_8-Pad8)
- J2 pad 9: Net-(J2-Pad9) -> unconnected-(J2-Pin_9-Pad9)
- U1 pad 45: Net-(U1-Pad45) -> unconnected-(U1-PB14A-Pad45)
- U1 pad 47: Net-(U1-Pad47) -> unconnected-(U1-PB14-Pad47)
- U4 pad 17: Net-(U4-Pad17) -> unconnected-(U4-B1-Pad17)
- U9 pad 4: Net-(U9-Pad4) -> unconnected-(U9-NC-Pad4)
Routing:
- net +5V: track 194.5 -> 214.4 mm, vias 13 -> 16
- net +1V2: track 109.8 -> 102.3 mm
- net /AN3: track 29.2 -> 34.1 mm
- net /~{C07X}in: track 61.5 -> 60.7 mm
- net /TDO: track 88.1 -> 88.7 mm
- net GND: track 155.6 -> 155.7 mm, vias 259 -> 256
- net /TMS: vias 3 -> 2
- net (no net): vias 1 -> 0
Other:
- net class Default removed
- rule pad_to_mask_clearance: 0.05 -> 0.0762
- rule solder_mask_min_width: 0.1 -> 0.127
- board text added: "JLCJLCJLCJLC"
- board text removed: "4203B"
- board text removed: "8 MB RAM"
- board text removed: "GW"
- board text removed: "Garrett’s Workshop"
- board text removed: "for Apple IIe"

Commit message: Change BOM to separate U4 from U3 and U5
Parts:
- U3, U5: value 74LVC245APW -> 74AHC245PW
Changed lines of the file:
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@@
     (descr "20-Lead Plastic Thin Shrink Small Outline (ST)-4.4 mm Body [TSSOP] (see Microchip Packaging Specification 00000049BS.pdf)")
     (tags "SSOP 0.65")
-    (property "LCSC Part" "C6082")
+    (property "LCSC Part" "C5516")
     (property "Mfg. Part Numbers" "NXP 74LVC245APW, TI SN74LVC245APW, NXP 74AHC245PW, NXP 74AHC245APW, TI 74AHC245PW")
     (property "Notes" "Most 74LVC245 or 74AHC245 in TSSOP-20 package is acceptable.")
@@
         (effects (font (size 0.8128 0.8128) (thickness 0.2032)))
     )
-    (fp_text value "74LVC245APW" (at 0 1.016 180) (layer "F.Fab")
+    (fp_text value "74AHC245PW" (at 0 1.016 180) (layer "F.Fab")
         (effects (font (size 0.508 0.508) (thickness 0.127)))
     )
@@
     (descr "20-Lead Plastic Thin Shrink Small Outline (ST)-4.4 mm Body [TSSOP] (see Microchip Packaging Specification 00000049BS.pdf)")
     (tags "SSOP 0.65")
-    (property "LCSC Part" "C6082")
+    (property "LCSC Part" "C5516")
     (property "Mfg. Part Numbers" "NXP 74LVC245APW, TI SN74LVC245APW, NXP 74AHC245PW, NXP 74AHC245APW, TI 74AHC245PW")
     (property "Notes" "Most 74LVC245 or 74AHC245 in TSSOP-20 package is acceptable.")
@@
         (effects (font (size 0.8128 0.8128) (thickness 0.2032)))
     )
-    (fp_text value "74LVC245APW" (at 0 1.016 180) (layer "F.Fab")
+    (fp_text value "74AHC245PW" (at 0 1.016 180) (layer "F.Fab")
         (effects (font (size 0.508 0.508) (thickness 0.127)))
     )
