File: Hardware/LCMXO2/RAM2E.kicad_pcb (KiCad board)
At the start: 4 copper layers, 78.2 x 50 mm, 79 parts, among them J1 AppleIIeAux, J2 microUSB, J3 C14M, J4 C14M, J5 JTAG, U1 LCMXO2-640-TG100, U10 CH340G, U11 74AHCT1G125GW, U2 W9812G6KH-6, U3 74AHC245PW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

Commit message: RC
Fix board IDs
Parts:
- R6: value 10k -> 2k2
- U1: value LCMXO2-640-TG100 -> LCMXO2-640HC-4TG100C
- U9: value AP2127K-1.8TRG1 -> AP2127K-1.2TRG1
Connections:
- U10 pad 11: +3V3 -> GND
- U10 pad 12: GND -> +3V3

Commit message: RC
Parts:
- added R14: 2k2, stdpads:R_0603, F.Cu at (259.6, 115.5)
- added R15: 2k2, stdpads:R_0603, F.Cu at (259.6, 117.0)
Routing:
- net /V~{OE}: track 19.1 -> 31.0 mm, vias 0 -> 2
- net /D~{OE}: track 21.5 -> 26.4 mm, vias 0 -> 2
- net +3V3: track 150.0 -> 151.5 mm, vias 91 -> 93
- net /R~{W}in: track 61.1 -> 60.4 mm
