File: Hardware/LCMXO2/RAM2E.kicad_pcb (KiCad board)
At the start: 4 copper layers, 78.2 x 50 mm, 81 parts, among them J1 AppleIIeAux, J2 microUSB, J3 C14M, J4 C14M, J5 JTAG, U1 LCMXO2-640HC-4TG100C, U10 CH340G, U11 74AHCT1G125GW, U2 W9812G6KH-6, U3 74AHC245PW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

Commit message: RC
Parts:
- U3, U5: value 74AHC245PW -> 74LVC245APW
Other:
- board text added: "C10C"
- board text removed: "B21C"

Commit message: RC
Parts:
- C29: value 2u2 -> 10u; footprint stdpads:C_0603 -> stdpads:C_0805
Changed lines of the file:
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@@
       (net 2 "GND") (pinfunction "1") (pintype "input") (zone_connect 2))
   )
-  (footprint "stdpads:C_0603" (layer "F.Cu")
+  (footprint "stdpads:C_0805" (layer "F.Cu")
     (at 269.875 126.238 180)
     (tags "capacitor")
-    (property "LCSC Part" "C23630")
+    (property "LCSC Part" "C15850")
     (property "Sheetfile" "RAM2E.kicad_sch")
     (property "Sheetname" "")
@@
     (property "ki_keywords" "capacitor cap")
     (solder_mask_margin 0.05)
-    (solder_paste_margin -0.04)
+    (solder_paste_margin -0.025)
     (attr smd)
-    (fp_text reference "C29" (at 0 0 180) (layer "F.Fab")
+    (fp_text reference "C29" (at 0 0) (layer "F.Fab")
         (effects (font (size 0.254 0.254) (thickness 0.0635)))
     )
-    (fp_text value "2u2" (at 0 0.25 180) (layer "F.Fab")
-        (effects (font (size 0.127 0.127) (thickness 0.03175)))
+    (fp_text value "10u" (at 0 0.35 180) (layer "F.Fab")
+        (effects (font (size 0.254 0.254) (thickness 0.0635)))
     )
-    (fp_text user "${REFERENCE}" (at 0 0 180) (layer "F.SilkS") hide
+    (fp_text user "${REFERENCE}" (at 0 0) (layer "F.SilkS") hide
         (effects (font (size 0.254 0.254) (thickness 0.0635)))
     )
-    (fp_line (start -0.162779 -0.51) (end 0.162779 -0.51)
-      (stroke (width 0.12) (type solid)) (layer "F.SilkS"))
-    (fp_line (start -0.162779 0.51) (end 0.162779 0.51)
-      (stroke (width 0.12) (type solid)) (layer "F.SilkS"))
-    (fp_line (start -1.4 -0.7) (end 1.4 -0.7)
+    (fp_line (start -0.4064 -0.8) (end 0.4064 -0.8)
+      (stroke (width 0.1524) (type solid)) (layer "F.SilkS"))
+    (fp_line (start -0.4064 0.8) (end 0.4064 0.8)
+      (stroke (width 0.1524) (type solid)) (layer "F.SilkS"))
+    (fp_line (start -1.7 -1) (end 1.7 -1)
       (stroke (width 0.05) (type solid)) (layer "F.CrtYd"))
-    (fp_line (start -1.4 0.7) (end -1.4 -0.7)
+    (fp_line (start -1.7 1) (end -1.7 -1)
       (stroke (width 0.05) (type solid)) (layer "F.CrtYd"))
-    (fp_line (start 1.4 -0.7) (end 1.4 0.7)
+    (fp_line (start 1.7 -1) (end 1.7 1)
       (stroke (width 0.05) (type solid)) (layer "F.CrtYd"))
-    (fp_line (start 1.4 0.7) (end -1.4 0.7)
+    (fp_line (start 1.7 1) (end -1.7 1)
       (stroke (width 0.05) (type solid)) (layer "F.CrtYd"))
-    (fp_line (start -0.8 -0.4) (end 0.8 -0.4)
-      (stroke (width 0.1) (type solid)) (layer "F.Fab"))
-    (fp_line (start -0.8 0.4) (end -0.8 -0.4)
-      (stroke (width 0.1) (type solid)) (layer "F.Fab"))
-    (fp_line (start 0.8 -0.4) (end 0.8 0.4)
-      (stroke (width 0.1) (type solid)) (layer "F.Fab"))
-    (fp_line (start 0.8 0.4) (end -0.8 0.4)
-      (stroke (width 0.1) (type solid)) (layer "F.Fab"))
-    (pad "1" smd roundrect (at -0.75 0 180) (size 0.85 0.95) (layers "F.Cu" "F.Paste" "F.Mask") (roundrect_rratio 0.25)
+    (fp_line (start -1 -0.625) (end 1 -0.625)
+      (stroke (width 0.15) (type solid)) (layer "F.Fab"))
+    (fp_line (start -1 0.625) (end -1 -0.625)
+      (stroke (width 0.15) (type solid)) (layer "F.Fab"))
+    (fp_line (start 1 -0.625) (end 1 0.625)
+      (stroke (width 0.15) (type solid)) (layer "F.Fab"))
+    (fp_line (start 1 0.625) (end -1 0.625)
+      (stroke (width 0.15) (type solid)) (layer "F.Fab"))
+    (pad "1" smd roundrect (at -0.85 0 180) (size 1.05 1.4) (layers "F.Cu" "F.Paste" "F.Mask") (roundrect_rratio 0.25)
       (net 1 "+5V") (pintype "passive"))
-    (pad "2" smd roundrect (at 0.75 0 180) (size 0.85 0.95) (layers "F.Cu" "F.Paste" "F.Mask") (roundrect_rratio 0.25)
+    (pad "2" smd roundrect (at 0.85 0 180) (size 1.05 1.4) (layers "F.Cu" "F.Paste" "F.Mask") (roundrect_rratio 0.25)
       (net 2 "GND") (pintype "passive"))
-    (model "${KICAD6_3DMODEL_DIR}/Capacitor_SMD.3dshapes/C_0603_1608Metric.wrl"
+    (model "${KICAD6_3DMODEL_DIR}/Capacitor_SMD.3dshapes/C_0805_2012Metric.wrl"
       (offset (xyz 0 0 0))
       (scale (xyz 1 1 1))
@@
     (pad "2" smd roundrect (at 0.95 0 90) (size 0.85 1.4) (layers "F.Cu" "F.Paste" "F.Mask") (roundrect_rratio 0.25)
       (net 158 "+1V2") (pintype "passive"))
+    (model "${KICAD6_3DMODEL_DIR}/Resistor_SMD.3dshapes/R_0805_2012Metric.wrl"
+      (offset (xyz 0 0 0))
+      (scale (xyz 1 1 1))
+      (rotate (xyz 0 0 0))
+    )
   )
   (footprint "stdpads:R_0603" (layer "F.Cu")
@@
     (pad "2" smd roundrect (at 0.8 0) (size 0.7 0.95) (layers "F.Cu" "F.Paste" "F.Mask") (roundrect_rratio 0.25)
       (net 141 "/~{INIT}") (pintype "passive"))
-    (model "${KICAD6_3DMODEL_DIR}/Resistor_SMD.3dshapes/R_0603_1608Metric.wrl"
-      (offset (xyz 0 0 0))
-      (scale (xyz 1 1 1))
-      (rotate (xyz 0 0 0))
-    )
   )
   (footprint "stdpads:R_0603" (layer "F.Cu")
@@
     (pad "2" smd roundrect (at 0.8 0) (size 0.7 0.95) (layers "F.Cu" "F.Paste" "F.Mask") (roundrect_rratio 0.25)
       (net 140 "/DONE") (pintype "passive"))
-    (model "${KICAD6_3DMODEL_DIR}/Resistor_SMD.3dshapes/R_0603_1608Metric.wrl"
-      (offset (xyz 0 0 0))
-      (scale (xyz 1 1 1))
-      (rotate (xyz 0 0 0))
-    )
   )
   (footprint "stdpads:Crystal_SMD_3225-4Pin_3.2x2.5mm" (layer "F.Cu")
@@
     (pad "5" smd roundrect (at -0.95 -1.05 180) (size 1.35 0.65) (layers "F.Cu" "F.Paste" "F.Mask") (roundrect_rratio 0.25)
       (net 158 "+1V2") (pinfunction "VOUT") (pintype "power_out"))
-    (model "${KICAD6_3DMODEL_DIR}/Package_TO_SOT_SMD.3dshapes/SOT-23-5.wrl"
-      (offset (xyz 0 0 0))
-      (scale (xyz 1 1 1))
-      (rotate (xyz 0 0 -90))
-    )
   )
   (footprint "stdpads:SOIC-16_3.9mm" (layer "F.Cu")
@@
     (solder_paste_margin -0.05)
     (attr smd)
-    (fp_text reference "R14" (at 0 0) (layer "F.Fab")
+    (fp_text reference "R14" (at 0 0 180) (layer "F.Fab")
         (effects (font (size 0.254 0.254) (thickness 0.0635)))
     )
-    (fp_text value "2k2" (at 0 0.25) (layer "F.Fab")
+    (fp_text value "2k2" (at 0 0.25 180) (layer "F.Fab")
         (effects (font (size 0.127 0.127) (thickness 0.03175)))
     )
-    (fp_text user "${REFERENCE}" (at 0 0) (layer "F.SilkS") hide
+    (fp_text user "${REFERENCE}" (at 0 0 180) (layer "F.SilkS") hide
         (effects (font (size 0.254 0.254) (thickness 0.0635)))
     )
@@
     (pad "2" smd roundrect (at 0.75 0 180) (size 0.85 0.95) (layers "F.Cu" "F.Paste" "F.Mask") (roundrect_rratio 0.25)
       (net 2 "GND") (pintype "passive"))
-    (model "${KICAD6_3DMODEL_DIR}/Capacitor_SMD.3dshapes/C_0603_1608Metric.wrl"
-      (offset (xyz 0 0 0))
-      (scale (xyz 1 1 1))
-      (rotate (xyz 0 0 0))
-    )
   )
   (footprint "stdpads:R_0603" (layer "F.Cu")
@@
     (solder_paste_margin -0.05)
     (attr smd)
-    (fp_text reference "R15" (at 0 0) (layer "F.Fab")
+    (fp_text reference "R15" (at 0 0 180) (layer "F.Fab")
         (effects (font (size 0.254 0.254) (thickness 0.0635)))
     )
-    (fp_text value "2k2" (at 0 0.25) (layer "F.Fab")
+    (fp_text value "2k2" (at 0 0.25 180) (layer "F.Fab")
         (effects (font (size 0.127 0.127) (thickness 0.03175)))
     )
-    (fp_text user "${REFERENCE}" (at 0 0) (layer "F.SilkS") hide
+    (fp_text user "${REFERENCE}" (at 0 0 180) (layer "F.SilkS") hide
         (effects (font (size 0.254 0.254) (thickness 0.0635)))
     )
@@
       (polygon
         (pts
-          (xy 204.851 123.571)
-          (xy 209.931 123.571)
-          (xy 209.931 122.301)
-          (xy 204.851 122.301)
+          (xy 204.724 123.698)
+          (xy 210.058 123.698)
+          (xy 210.058 122.174)
+          (xy 204.724 122.174)
         )
       )
