File: Hardware/LCMXO2/Docs.kicad_sch (KiCad schematic)
At the start: 0 parts

Commit message: RC
Other:
- title: GW4203B (RAM2E II) - LCMXO2-640 / LCMXO2-1200 -> GW4203C (RAM2E II) - LCMXO2-640 / LCMXO2-1200
Changed lines of the file:
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@@
   (paper "A4")
   (title_block
-    (title "GW4203B (RAM2E II) - LCMXO2-640 / LCMXO2-1200")
-    (date "2024-04-24")
-    (rev "2.1")
+    (title "GW4203C (RAM2E II) - LCMXO2-640 / LCMXO2-1200")
+    (date "2024-05-20")
+    (rev "1.0")
     (company "Garrett's Workshop")
   )
