File: Hardware/iCE40/RAM2E.kicad_pcb (KiCad board)
At the start: 4 copper layers, 78.2 x 50 mm, 66 parts, among them J1 AppleIIeAux, J2 JTAG, J3 C14M, U1 LCMXO256-TQFP-100, U2 W9812G6KH-6, U3 74LVC245APW, U4 74LVC245APW, U5 74LVC245APW, U6 74AHCT245PW, U7 74AHCT245PW, U8 XC6206P332MR, U9 AP2127K-1.8TRG1

Commit message: still workin
Parts:
- removed the C11 at (230.3, 107.3)
- removed the C29 at (246.3, 118.0)
- removed the C9 at (239.1, 118.0)
- removed REF**: SOIC-8_3.9mm, stdpads:SOIC-8_3.9mm
- removed RN1, RN2, RN3, RN4, RN5: 4x33, stdpads:R4_0402
- added C30: 2u2, stdpads:C_0603, F.Cu at (273.9, 99.2)
- added C31: 10u, stdpads:C_0805, F.Cu at (271.4, 115.7)
- added C32: 10u, stdpads:C_0805, F.Cu at (263.9, 115.7)
- added C33: 2u2, stdpads:C_0603, F.Cu at (237.3, 98.7)
- added C34: 2u2, stdpads:C_0603, F.Cu at (240.8, 98.7)
- added C35: 2u2, stdpads:C_0603, F.Cu at (230.3, 106.6)
- added C36: 2u2, stdpads:C_0603, F.Cu at (248.3, 98.7)
- added C37: 15p, stdpads:C_0603, F.Cu at (257.6, 103.8)
- added R11: 47, stdpads:R_0603, F.Cu at (228.2, 118.5)
- added R12: 47, stdpads:R_0603, F.Cu at (257.6, 101.0)
- added R4: 47, stdpads:R_0603, F.Cu at (204.3, 108.5)
- added R5: 1k, stdpads:R_0603, F.Cu at (256.4, 97.2)
- added R8: 10k, stdpads:R_0603, F.Cu at (207.4, 107.7)
- added U10: AP2127K-2.5TRG1, stdpads:SOT-23-5, F.Cu at (267.6, 115.5)
- added U11: 25F010, stdpads:SOIC-8_5.3mm, F.Cu at (268.0, 100.3)
- R1: value 0 -> 47; footprint stdpads:R_0805 -> stdpads:R_0603
- R10, R9: value 22k -> 10k; footprint stdpads:R_0805 -> stdpads:R_0603
- U1: value LCMXO256-TQFP-100 -> iCE40HX1K-VQ100
- U9: value AP2127K-1.8TRG1 -> AP2127K-1.2TRG1
- moved R9 54.1 mm to (257.6, 102.4)
- moved C17 45.5 mm to (245.3, 118.0), turned to 180 degrees
- moved C19 41.1 mm to (249.8, 108.6), turned to 90 degrees
- moved C18 37.7 mm to (249.8, 111.6), turned to 270 degrees
- moved R1 33.8 mm to (226.8, 118.5), turned to 270 degrees
- moved C13 18.0 mm to (230.3, 113.1), turned to 270 degrees
- moved C14 14.9 mm to (236.8, 118.0), turned to 0 degrees
- moved C15 12.7 mm to (240.3, 118.0), turned to 0 degrees
- moved C12 11.4 mm to (230.3, 109.6), turned to 270 degrees
- moved C16 9.77 mm to (244.8, 98.7), turned to 180 degrees
- moved C25 2.05 mm to (223.8, 118.0), turned to 0 degrees
- moved R10 1.15 mm to (207.4, 109.2)
- moved R3 0.50 mm to (229.7, 118.5)
- turned U1 to 270 degrees
Connections:
- net Net-(J2-Pad8) renamed /~INIT~
- C16 pad 1: +3V3 -> +1V2
- C19 pad 1: +1V8 -> +1V2
- C4 pad 1: +1V8 -> +1V2
- C5 pad 1: +1V8 -> +1V2
- J2 pad 1: /TCK -> /CCK
- J2 pad 10: GND -> /C~CS~
- J2 pad 3: /TDO -> /Mode
- J2 pad 4: +3V3 -> GND
- J2 pad 5: /TMS -> /CDI
- J2 pad 6: Net-(J2-Pad6) -> +3V3
- J2 pad 7: Net-(J2-Pad7) -> /CDO
- J2 pad 9: /TDI -> /C~RST~
- R1 pad 1: +3V3 -> /RCLK
- R1 pad 2: +1V8 -> Net-(R1-Pad2)
- R10 pad 2: /TMS -> /C~CS~
- R9 pad 1: /TCK -> +3V3
- R9 pad 2: GND -> /CCKr
- U1 pad 1: /~EN80~in -> /~WE~
- U1 pad 10: +3V3 -> /RA0
- U1 pad 100: /~WE~ -> /DQMH
- U1 pad 11: /Ain1 -> +1V2
- U1 pad 12: GND -> /RA7
- U1 pad 13: /Ain7 -> /ACLK
- U1 pad 14: /~C07X~in -> +3V3
- U1 pad 15: /R~W~in -> /RA1
- U1 pad 16: /Din7 -> /RA6
- U1 pad 17: /Din6 -> GND
- U1 pad 18: /Din0 -> /RA2
- U1 pad 19: /Din1 -> /RA8
- U1 pad 2: /Ain2 -> /BA0
- U1 pad 20: /Din3 -> /RA5
- U1 pad 21: /Din2 -> /RA3
- U1 pad 22: /Din4 -> +3V3
- U1 pad 23: /Din5 -> GND
- U1 pad 24: +3V3 -> /RA4
- U1 pad 25: GND -> /~EN80~in
- U1 pad 26: /TDO -> /R~W~80in
- U1 pad 27: Net-(U1-Pad27) -> /Ain5
- U1 pad 28: /TMS -> /PHI1in
- U1 pad 29: Net-(U1-Pad29) -> /Ain6
- U1 pad 3: /R~W~80in -> /~CAS~
- U1 pad 30: Net-(U1-Pad30) -> /Ain7
- U1 pad 31: /TDI -> +3V3
- U1 pad 32: Net-(U1-Pad32) -> GND
- U1 pad 33: /TCK -> /Ain0
- U1 pad 34: Net-(U1-Pad34) -> /Din7
- U1 pad 36: Net-(U1-Pad36) -> /Din6
- U1 pad 37: Net-(U1-Pad37) -> /Ain4
- U1 pad 38: Net-(U1-Pad38) -> +3V3
- U1 pad 39: Net-(U1-Pad39) -> GND
- U1 pad 4: /Ain4 -> /RA11
- U1 pad 40: GND -> /Ain1
- U1 pad 41: +3V3 -> /Din0
- U1 pad 42: GND -> /Din1
- U1 pad 43: Net-(U1-Pad43) -> /CDONE
- U1 pad 44: Net-(U1-Pad44) -> /C~RST~
- U1 pad 45: Net-(U1-Pad45) -> /CDO
- U1 pad 46: Net-(U1-Pad46) -> /CDI
- U1 pad 47: Net-(U1-Pad47) -> GND
- U1 pad 48: GND -> /CCKr
- U1 pad 49: Net-(U1-Pad49) -> /C~CS~
- U1 pad 5: /Ain5 -> GND
- U1 pad 50: Net-(U1-Pad50) -> +3V3
- U1 pad 51: Net-(U1-Pad51) -> /Din2
- U1 pad 52: Net-(U1-Pad52) -> /Din5
- U1 pad 53: Net-(U1-Pad53) -> /Vout7
- U1 pad 54: Net-(U1-Pad54) -> /Vout3
- U1 pad 55: Net-(U1-Pad55) -> GND
- U1 pad 56: Net-(U1-Pad56) -> /Ain2
- U1 pad 57: Net-(U1-Pad57) -> /Din3
- U1 pad 58: Net-(U1-Pad58) -> +3V3
- U1 pad 59: Net-(U1-Pad59) -> /Ain3
- U1 pad 6: /Ain3 -> +3V3
- U1 pad 60: +3V3 -> /Vout6
- U1 pad 61: Net-(U1-Pad61) -> +1V2
- U1 pad 62: GND -> /Din4
- U1 pad 63: Net-(U1-Pad63) -> /R~W~in
- U1 pad 64: Net-(U1-Pad64) -> /~C07X~in
- U1 pad 65: Net-(U1-Pad65) -> /Vout1
- U1 pad 66: Net-(U1-Pad66) -> /Vout5
- U1 pad 67: Net-(U1-Pad67) -> +3V3
- U1 pad 68: Net-(U1-Pad68) -> /Vout2
- U1 pad 69: Net-(U1-Pad69) -> /Vout0
- U1 pad 7: /PHI1in -> /BA1
- U1 pad 70: Net-(U1-Pad70) -> GND
- U1 pad 71: Net-(U1-Pad71) -> /Vout4
- U1 pad 72: /DQMH -> /D~OE~
- U1 pad 73: /DQML -> /Dout5
- U1 pad 74: +3V3 -> /Dout4
- U1 pad 75: GND -> +2V5
- U1 pad 76: /RA4 -> Net-(U1-Pad76)
- U1 pad 77: /RA6 -> +1V2
- U1 pad 78: /RA1 -> /Dout3
- U1 pad 79: /RA7 -> /Dout2
- U1 pad 8: /Ain6 -> /RA9
- U1 pad 80: /RA0 -> /Dout1
- U1 pad 81: /RA8 -> /Dout0
- U1 pad 82: /RA10 -> /Dout6
- U1 pad 83: /RA9 -> /Dout7
- U1 pad 85: /BA1 -> /RD0
- U1 pad 86: /ACLK -> /RD1
- U1 pad 87: /RA3 -> /RD2
- U1 pad 89: /RA2 -> /RD3
- U1 pad 9: /Ain0 -> /RA10
- U1 pad 90: +1V2 -> /RD4
- U1 pad 91: /RA5 -> /RD5
- U1 pad 93: GND -> /RD6
- U1 pad 94: /~CS~ -> /RD7
- U1 pad 95: /RA11 -> /~RAS~
- U1 pad 96: /BA0 -> /DQML
- U1 pad 97: /~RAS~ -> /~CS~
- U1 pad 98: /CKE -> GND
- U1 pad 99: /~CAS~ -> /CKE
- U3 pad 11: Net-(RN5-Pad4) -> /Ain3
- U3 pad 12: Net-(RN5-Pad3) -> /Ain4
- U3 pad 13: Net-(RN5-Pad2) -> /Ain2
- U3 pad 14: Net-(RN5-Pad1) -> /Ain0
- U3 pad 15: Net-(RN4-Pad4) -> /Ain1
- U3 pad 16: Net-(RN4-Pad3) -> /Ain7
- U3 pad 17: Net-(RN4-Pad2) -> /~C07X~in
- U3 pad 18: Net-(RN4-Pad1) -> /R~W~in
- U4 pad 18: Net-(RN3-Pad1) -> Net-(R1-Pad2)
- U6 pad 19: /V~OE~ -> /PHI1
- U9 pad 5: +1V8 -> +1V2
Routing:
- net /CDI: track 0.00 -> 153.3 mm, vias 0 -> 4
- net /CDO: track 0.00 -> 127.0 mm, vias 0 -> 4
- net /C~CS~: track 0.00 -> 113.9 mm, vias 0 -> 5
- net /C~RST~: track 0.00 -> 110.5 mm, vias 0 -> 4
- net /CCKr: track 0.00 -> 107.8 mm, vias 0 -> 3
- net /TDO: track 96.4 -> 0.00 mm, vias 2 -> 0
- net /TMS: track 92.1 -> 0.00 mm, vias 3 -> 0
- net /TDI: track 76.6 -> 0.00 mm, vias 2 -> 0
- net +2V5: track 0.00 -> 72.9 mm, vias 0 -> 6
- net +1V2: track 33.1 -> 98.0 mm, vias 3 -> 7
- net /TCK: track 61.1 -> 0.00 mm, vias 2 -> 0
- net +5V: track 194.6 -> 237.0 mm, vias 13 -> 16
- net /Dout7: track 0.95 -> 41.9 mm
- net /Dout6: track 1.15 -> 40.8 mm
- net /Dout0: track 1.35 -> 39.7 mm
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- added copper zone on F.Cu, net +1V2
- removed copper zone on F.Cu, net +1V8
Other:
- board text added: "20D"

Commit message: Generated gerbers and documentation
Parts:
- added D1: White, stdpads:LED_0805, F.Cu at (229.5, 98.8)
- added R13: 180, stdpads:R_0805, F.Cu at (229.5, 100.8)
- added U12: 74LVC1G97, stdpads:SOT-363, F.Cu at (263.5, 128.5)
- R5: value 1k -> 10k
- moved R5 5.46 mm to (254.7, 102.4)
Connections:
- U1 pad 72: /D~OE~ -> /LED
Routing:
- net /LED: track 0.00 -> 44.1 mm, vias 0 -> 2
- net +2V5: track 72.9 -> 99.1 mm
- net /D~OE~: track 22.1 -> 12.9 mm
- net /CDONE: track 27.4 -> 23.2 mm
- net +3V3: track 135.3 -> 138.1 mm, vias 90 -> 93
- net /R~W~80: track 44.5 -> 47.0 mm, vias 1 -> 2
- net /C~CS~: track 113.9 -> 111.5 mm
- net Net-(D1-Pad2): track 0.00 -> 1.96 mm
- net /PHI1: track 62.6 -> 61.0 mm
- net /C~RST~: track 110.5 -> 109.3 mm
- net /CDI: track 153.3 -> 152.3 mm
- net GND: track 174.9 -> 175.9 mm, vias 253 -> 257
- net /~EN80~: track 49.8 -> 49.2 mm
- net /CCKr: track 107.8 -> 108.4 mm
Other:
- board text added: "B20D"
- board text removed: "20D"
