File: Hardware/iCE40/RAM2E.sch (KiCad schematic (older format))
At the start: 62 parts, among them J1 AppleIIeAux, J2 JTAG, J3 C14M, U2 W9812G6KH-6, U3 74LVC245APW, U4 74LVC245APW, U5 74LVC245APW, U6 74AHCT245PW, U7 74AHCT245PW, U8 XC6206P332MR, U9 AP2127K-1.2TRG1

Commit message: still workin
Parts:
- removed RN1, RN2, RN3, RN4, RN5: 4x33, stdpads:R4_0402, symbol Device:R_Pack04
- removed U?: iCE40HX1K-VQ100, stdpads:TQFP-100, symbol GW_PLD:iCE40HX1K-VQ100
- added C30, C33, C34, C35, C36: 2u2, stdpads:C_0603, symbol Device:C_Small
- added C31, C32: 10u, stdpads:C_0805, symbol Device:C_Small
- added C37: 15p, stdpads:C_0603, symbol Device:C_Small
- added R11, R12, R4: 47, stdpads:R_0603, symbol Device:R_Small
- added R5: 1k, stdpads:R_0603, symbol Device:R_Small
- added R9: 10k, stdpads:R_0603, symbol Device:R_Small
- added U1: iCE40HX1K-VQ100, stdpads:TQFP-100_14x14mm_P0.5mm, symbol GW_PLD:iCE40HX1K-VQ100
- added U10: AP2127K-2.5TRG1, stdpads:SOT-23-5, symbol Regulator_Linear:AP2127K-2.5
- added U11: 25F010, stdpads:SOIC-8_5.3mm, symbol GW_RAM:SPIFlash-SO-8
- R1: value 0 -> 47; footprint stdpads:R_0805 -> stdpads:R_0603; LCSC Part C17477 -> C23182; Mfg. Part Numbers Uniroyal 0805W8F2202T5E -> Uniroyal 0603WAF470JT5E
- R10: value 22k -> 10k; footprint stdpads:R_0805 -> stdpads:R_0603
- R8: renamed from R9; value 22k -> 10k; footprint stdpads:R_0805 -> stdpads:R_0603
Connections:
- net +1V2: now also C35.1, U1.11 (Vcc), U1.35 (Vcc), U1.61 (Vcc), U1.77 (Vcc); no longer R1.2
- net +2V5: now also C32.1, C36.1, U1.75 (Vpp2V5), U10.5 (VOUT)
- net +3V3: now also J2.6 (Pin_6), R8.1, C30.1, C33.1, C34.1, R5.1, R9.1, U1.14 (VccIO3), U1.22 (VccIO3), U1.31 (VccIO2), U1.38 (VccIO2), U1.50 (VccSPI), U1.58 (VccIO1), U1.6 (VccIO3), U1.67 (VccIO1), U1.88 (VccIO0), U1.92 (VccIO0), U11.3 (~WP~/IO2), U11.7 (~HLD~/IO3), U11.8 (Vcc); no longer J2.4 (Pin_4), R1.1
- net +5V: now also C31.1, U10.1 (VIN), U10.3 (EN)
- net ACLK: now also R11.1, U1.13 (IOL_6B_GBIN7)
- net Ain0: now also U3.14 (B4), U1.33 (IOB_35_GBIN5)
- net Ain1: now also U3.15 (B3), U1.40 (IOB_41)
- net Ain2: now also U3.13 (B5), U1.56 (IOR_56)
- net Ain3: now also U3.11 (B7), U1.59 (IOR_58)
- net Ain4: now also U3.12 (B6), U1.37 (IOB_37)
- net Ain5: now also U1.27 (IOB_27)
- net Ain6: now also U1.29 (IOB_29)
- net Ain7: now also U3.16 (B2), U1.30 (IOB_30)
- net BA0: now also U1.2 (IOL_1B)
- net BA1: now also U1.7 (IOL_3A)
- net CKE: now also U1.99 (IOT_93)
- net DQMH: now also U1.100 (IOT_95)
- net DQML: now also U1.96 (IOT_90)
- net Din0: now also U1.41 (IOB_42_CBSEL0)
- net Din1: now also U1.42 (IOB_43_CBSEL1)
- net Din2: now also U1.51 (IOR_52)
- net Din3: now also U1.57 (IOR_57)
- net Din4: now also U1.62 (IOR_60_GBIN3)
- net Din5: now also U1.52 (IOR_53)
- net Din6: now also U1.36 (IOB_34)
- net Din7: now also U1.34 (IOB_36_GBIN4)
- net Dout0: now also U1.81 (IOT_77)
- net Dout1: now also U1.80 (IOT_75)
- net Dout2: now also U1.79 (IOT_74)
- net Dout3: now also U1.78 (IOT_73)
- net Dout4: now also U1.74 (IOR_72)
- net Dout5: now also U1.73 (IOR_71)
- net Dout6: now also U1.82 (IOT_78)
- net Dout7: now also U1.83 (IOT_79)
- net D~OE~: now also U1.72 (IOR_70)
- net GND: now also J2.4 (Pin_4), C30.2, C31.2, C32.2, C33.2, C34.2, C35.2, C36.2, C37.2, U1.17 (GND), U1.23 (GND), U1.32 (GND), U1.39 (GND), U1.47 (GND), U1.5 (GND), U1.55 (GND), U1.70 (GND), U1.84 (GND), U1.98 (GND), U10.2 (GND), U11.4 (GND); no longer J2.10 (Pin_10), R8.2
- net PHI1in: now also U1.28 (IOB_28)
- net RA0: now also U1.10 (IOL_5B)
- net RA1: now also U1.15 (IOL_7A_GBIN6)
- net RA10: now also U1.9 (IOL_5A)
- net RA11: now also U1.4 (IOL_2B)
- net RA2: now also U1.18 (IOL_8A)
- net RA3: now also U1.21 (IOL_10B)
- net RA4: now also U1.24 (IOL_12A)
- net RA5: now also U1.20 (IOL_10A)
- net RA6: now also U1.16 (IOL_7B)
- net RA7: now also U1.12 (IOL_6A)
- net RA8: now also U1.19 (IOL_8B)
- net RA9: now also U1.8 (IOL_3B)
- net RCLK: now also R1.1
- net RD0: now also U1.85 (IOT_80)
- net RD1: now also U1.86 (IOT_81)
- net RD2: now also U1.87 (IOT_82)
- net RD3: now also U1.89 (IOT_84_GBIN1)
- net RD4: now also U1.90 (IOT_85_GBIN0)
- net RD5: now also U1.91 (IOT_86)
- net RD6: now also U1.93 (IOT_87)
- net RD7: now also U1.94 (IOT_88)
- net R~W~80in: now also U1.26 (IOB_26)
- net R~W~in: now also U3.18 (B0), U1.63 (IOR_61_GBIN2)
- net Vout0: now also U1.69 (IOR_68)
- net Vout1: now also U1.65 (IOR_64)
- net Vout2: now also U1.68 (IOR_67)
- net Vout3: now also U1.54 (IOR_55)
- net Vout4: now also U1.71 (IOR_69)
- net Vout5: now also U1.66 (IOR_65)
- net Vout6: now also U1.60 (IOR_59)
- net Vout7: now also U1.53 (IOR_54)
- net ~C07X~in: now also U3.17 (B1), U1.64 (IOR_63)
- net ~CAS~: now also U1.3 (IOL_2A)
- net ~CS~: now also U1.97 (IOT_91)
- net ~EN80~in: now also U1.25 (IOL_12B)
- net ~RAS~: now also U1.95 (IOT_89)
- net ~WE~: now also U1.1 (IOL_1A)
- net CDO: now reaches J2.7 (Pin_7)
- net CDO: now also U1.45 (IOB_44_SDO), U11.5 (DI/IO0)
- net ~INIT~: now reaches J2.8 (Pin_8)
- net at U4.18 (B0): now also R1.2, R11.2
- net TCK renamed CCK
- net CCK: now also R4.2; no longer R8.1
- net TDI renamed C~RST~
- net C~RST~: now also R8.2, U1.44 (~CRST~)
- net TDO renamed Mode
- net TMS renamed CDI
- net CDI: now also U1.46 (IOB_45_SDI), U11.2 (DO/IO1); no longer R10.2
- new net CCKr: C37.1, R12.2, R4.1, R9.2, U1.48 (IOB_46_SCK)
- new net CCKrF: R12.1, U11.6 (CLK)
- new net CDONE: R5.2, U1.43 (CDONE)
- new net C~CS~: J2.10 (Pin_10), R10.2, U1.49 (IOB_47_SS), U11.1 (~CS~)
- no-connect marks 9 -> 2
Other:
- moved on the sheet: C16, C19, J3, R10, R3

Commit message: Generated gerbers and documentation
Parts:
- added D1: White, stdpads:LED_0805, symbol Device:LED_Small_ALT
- added R13: 180, stdpads:R_0805, symbol Device:R_Small
- added U12: 74LVC1G97, stdpads:SOT-363, symbol 74xGxx:74LVC1G97
- C37: LCSC Part (none) -> C1644; Mfg. Part Numbers (none) -> Samsung CL10C150JB8NNNC; Notes (none) -> 10V or higher. Any manufacturer's part is acceptable but Sa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
- R10, R8, R9: LCSC Part C17560 -> C25804; Mfg. Part Numbers Uniroyal 0805W8F2202T5E -> Uniroyal 0603WAF1002T5E
- R5: value 1k -> 10k; LCSC Part C17560 -> C25804; Mfg. Part Numbers Uniroyal 0805W8F2202T5E -> Uniroyal 0603WAF1002T5E
- R6: Mfg. Part Numbers Uniroyal 0805W8F2202T5E -> Uniroyal 0805W8F0000T5E
- U1: LCSC Part (none) -> C1519043; Mfg. Part Numbers (none) -> Lattice iCE40HX1K-VQ100
- U10: LCSC Part (none) -> C460326; Mfg. Part Numbers (none) -> Diodes AP2127K-2.5TRG1, Torex XC6206J252MR; Notes (none) -> Most 2.5V regulator in SOT-23-5 package is acceptable.
- U11: LCSC Part (none) -> C2687406; Mfg. Part Numbers (none) -> Zetta ZD25WD20BTIGT, Adesto AT25SF081-SSHD, Winbond W25X20C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; Notes (none) -> Most SPI flash in SOIC-8 (3.9mm / 150 mil width) package is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
- U2: Notes Most 166 MHz 128/256 Mbit SDRAM is acceptable. -> Most 166 MHz 128/256 Mbit x16 SDRAM is acceptable.
- U3, U4, U5: Mfg. Part Numbers NXP 74LVC245APW, TI SN74LVC245APW -> NXP 74LVC245APW, TI SN74LVC245APW, NXP 74AHC245PW, NXP 74AH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; Notes (none) -> Most 74LVC245 or 74AHC245 in TSSOP-20 package is acceptable.
- U6, U7: Mfg. Part Numbers NXP 74AHCT245PW, TI SN74AHCT245PW -> NXP 74AHCT245PW, NXP 74AHCT245APW, TI SN74AHCT245PW; Notes (none) -> Most 74AHCT245 in TSSOP-20 package is acceptable.
- U8: Notes (none) -> Most 3.3V regulator in SOT-23 package is acceptable.
- U9: LCSC Part (none) -> C151376; Mfg. Part Numbers (none) -> Diodes AP2127K-1.2TRG1, Torex XC6228D122VR; Notes (none) -> Most 1.2V regulator in SOT-23-5 package is acceptable.
Connections:
- net +3V3: now also R13.2, U12.1 (IN1), U12.5 (VCC)
- net D~OE~: now also U12.4 (Y); no longer U1.72 (IOR_70)
- net GND: now also U12.2 (GND)
- net R~W~80: now also U12.6 (IN2)
- net ~EN80~: now also U12.3 (IN0)
- new net: D1.2 (A), R13.1
- new net LED: D1.1 (K), U1.72 (IOR_70)
